File: source/kicad/main/main.kicad_pcb (KiCad board)
At the start: 2 copper layers, 0 parts

Commit message: Add basic pcb placement; Add lcsc&pcb libs
Parts:
- added psu.configuration_resistors[0][Resistor:5.0KΩ]: 5.0KΩ, lcsc:R0402, F.Cu at (184.2, 123.3)
- added psu.configuration_resistors[1][Resistor:5.0KΩ]: 5.0KΩ, lcsc:R0402, F.Cu at (166.8, 136.5)
- added psu.usb[USB_C_Receptacle:x]: x, lcsc:USB-C-SMD_TYPE-C-USB-18, F.Cu at (167.6, 104.1)
- added tester.cc1.indicator.led.current_limiting_resistor[Resistor:R]: R, lcsc:R0402, F.Cu at (58.0, 15.0)
- added tester.cc1.indicator.led.led[LED:D]: D, lcsc:LED0805-R-RD, F.Cu at (62.0, 15.0)
- added tester.cc1.indicator.power_switch.mosfet[MOSFET:Q]: Q, lcsc:SOT-23-3_L2.9-W1.3-P1.90-LS2.4-BR, F.Cu at (54.0, 15.0)
- added tester.cc1.indicator.power_switch.pull_resistor[Resistor:R]: R, lcsc:R0402, F.Cu at (50.0, 15.0)
- added tester.cc2.indicator.led.current_limiting_resistor[Resistor:R]: R, lcsc:R0402, F.Cu at (58.0, 19.0)
- added tester.cc2.indicator.led.led[LED:D]: D, lcsc:LED0805-R-RD, F.Cu at (62.0, 19.0)
- added tester.cc2.indicator.power_switch.mosfet[MOSFET:Q]: Q, lcsc:SOT-23-3_L2.9-W1.3-P1.90-LS2.4-BR, F.Cu at (54.0, 19.0)
- added tester.cc2.indicator.power_switch.pull_resistor[Resistor:R]: R, lcsc:R0402, F.Cu at (50.0, 19.0)
- added tester.d1[0].indicator.led.current_limiting_resistor[Resistor:R]: R, lcsc:R0402, F.Cu at (58.0, 23.0)
- added tester.d1[0].indicator.led.led[LED:D]: D, lcsc:LED0805-R-RD, F.Cu at (62.0, 23.0)
- added tester.d1[0].indicator.power_switch.mosfet[MOSFET:Q]: Q, lcsc:SOT-23-3_L2.9-W1.3-P1.90-LS2.4-BR, F.Cu at (54.0, 23.0)
- added tester.d1[0].indicator.power_switch.pull_resistor[Resistor:R]: R, lcsc:R0402, F.Cu at (50.0, 23.0)
- added tester.d1[1].indicator.led.current_limiting_resistor[Resistor:R]: R, lcsc:R0402, F.Cu at (58.0, 27.0)
- added tester.d1[1].indicator.led.led[LED:D]: D, lcsc:LED0805-R-RD, F.Cu at (62.0, 27.0)
- added tester.d1[1].indicator.power_switch.mosfet[MOSFET:Q]: Q, lcsc:SOT-23-3_L2.9-W1.3-P1.90-LS2.4-BR, F.Cu at (54.0, 27.0)
- added tester.d1[1].indicator.power_switch.pull_resistor[Resistor:R]: R, lcsc:R0402, F.Cu at (50.0, 27.0)
- added tester.d2[0].indicator.led.current_limiting_resistor[Resistor:R]: R, lcsc:R0402, F.Cu at (58.0, 31.0)
- added tester.d2[0].indicator.led.led[LED:D]: D, lcsc:LED0805-R-RD, F.Cu at (62.0, 31.0)
- added tester.d2[0].indicator.power_switch.mosfet[MOSFET:Q]: Q, lcsc:SOT-23-3_L2.9-W1.3-P1.90-LS2.4-BR, F.Cu at (54.0, 31.0)
- added tester.d2[0].indicator.power_switch.pull_resistor[Resistor:R]: R, lcsc:R0402, F.Cu at (50.0, 31.0)
- added tester.d2[1].indicator.led.current_limiting_resistor[Resistor:R]: R, lcsc:R0402, F.Cu at (58.0, 35.0)
- added tester.d2[1].indicator.led.led[LED:D]: D, lcsc:LED0805-R-RD, F.Cu at (62.0, 35.0)
- added tester.d2[1].indicator.power_switch.mosfet[MOSFET:Q]: Q, lcsc:SOT-23-3_L2.9-W1.3-P1.90-LS2.4-BR, F.Cu at (54.0, 35.0)
- added tester.d2[1].indicator.power_switch.pull_resistor[Resistor:R]: R, lcsc:R0402, F.Cu at (50.0, 35.0)
- added tester.gnd[0].indicator.led.current_limiting_resistor[Resistor:R]: R, lcsc:R0402, F.Cu at (58.0, 39.0)
- added tester.gnd[0].indicator.led.led[LED:D]: D, lcsc:LED0805-R-RD, F.Cu at (62.0, 39.0)
- added tester.gnd[0].indicator.power_switch.mosfet[MOSFET:Q]: Q, lcsc:SOT-23-3_L2.9-W1.3-P1.90-LS2.4-BR, F.Cu at (54.0, 39.0)
- added tester.gnd[0].indicator.power_switch.pull_resistor[Resistor:R]: R, lcsc:R0402, F.Cu at (50.0, 39.0)
- added tester.gnd[1].indicator.led.current_limiting_resistor[Resistor:R]: R, lcsc:R0402, F.Cu at (58.0, 43.0)
- added tester.gnd[1].indicator.led.led[LED:D]: D, lcsc:LED0805-R-RD, F.Cu at (62.0, 43.0)
- added tester.gnd[1].indicator.power_switch.mosfet[MOSFET:Q]: Q, lcsc:SOT-23-3_L2.9-W1.3-P1.90-LS2.4-BR, F.Cu at (54.0, 43.0)
- added tester.gnd[1].indicator.power_switch.pull_resistor[Resistor:R]: R, lcsc:R0402, F.Cu at (50.0, 43.0)
- added tester.gnd[2].indicator.led.current_limiting_resistor[Resistor:R]: R, lcsc:R0402, F.Cu at (58.0, 47.0)
- added tester.gnd[2].indicator.led.led[LED:D]: D, lcsc:LED0805-R-RD, F.Cu at (62.0, 47.0)
- added tester.gnd[2].indicator.power_switch.mosfet[MOSFET:Q]: Q, lcsc:SOT-23-3_L2.9-W1.3-P1.90-LS2.4-BR, F.Cu at (54.0, 47.0)
- added tester.gnd[2].indicator.power_switch.pull_resistor[Resistor:R]: R, lcsc:R0402, F.Cu at (50.0, 47.0)
- added tester.gnd[3].indicator.led.current_limiting_resistor[Resistor:R]: R, lcsc:R0402, F.Cu at (58.0, 51.0)
- added tester.gnd[3].indicator.led.led[LED:D]: D, lcsc:LED0805-R-RD, F.Cu at (62.0, 51.0)
- added tester.gnd[3].indicator.power_switch.mosfet[MOSFET:Q]: Q, lcsc:SOT-23-3_L2.9-W1.3-P1.90-LS2.4-BR, F.Cu at (54.0, 51.0)
- added tester.gnd[3].indicator.power_switch.pull_resistor[Resistor:R]: R, lcsc:R0402, F.Cu at (50.0, 51.0)
- added tester.pair1_rx1[0].indicator.led.current_limiting_resistor[Resistor:R]: R, lcsc:R0402, F.Cu at (58.0, 55.0)
- added tester.pair1_rx1[0].indicator.led.led[LED:D]: D, lcsc:LED0805-R-RD, F.Cu at (62.0, 55.0)
- added tester.pair1_rx1[0].indicator.power_switch.mosfet[MOSFET:Q]: Q, lcsc:SOT-23-3_L2.9-W1.3-P1.90-LS2.4-BR, F.Cu at (54.0, 55.0)
- added tester.pair1_rx1[0].indicator.power_switch.pull_resistor[Resistor:R]: R, lcsc:R0402, F.Cu at (50.0, 55.0)
- added tester.pair1_rx1[1].indicator.led.current_limiting_resistor[Resistor:R]: R, lcsc:R0402, F.Cu at (58.0, 59.0)
- added tester.pair1_rx1[1].indicator.led.led[LED:D]: D, lcsc:LED0805-R-RD, F.Cu at (62.0, 59.0)
- added tester.pair1_rx1[1].indicator.power_switch.mosfet[MOSFET:Q]: Q, lcsc:SOT-23-3_L2.9-W1.3-P1.90-LS2.4-BR, F.Cu at (54.0, 59.0)
- added tester.pair1_rx1[1].indicator.power_switch.pull_resistor[Resistor:R]: R, lcsc:R0402, F.Cu at (50.0, 59.0)
- added tester.pair2_rx2[0].indicator.led.current_limiting_resistor[Resistor:R]: R, lcsc:R0402, F.Cu at (58.0, 63.0)
- added tester.pair2_rx2[0].indicator.led.led[LED:D]: D, lcsc:LED0805-R-RD, F.Cu at (62.0, 63.0)
- added tester.pair2_rx2[0].indicator.power_switch.mosfet[MOSFET:Q]: Q, lcsc:SOT-23-3_L2.9-W1.3-P1.90-LS2.4-BR, F.Cu at (54.0, 63.0)
- added tester.pair2_rx2[0].indicator.power_switch.pull_resistor[Resistor:R]: R, lcsc:R0402, F.Cu at (50.0, 63.0)
- added tester.pair2_rx2[1].indicator.led.current_limiting_resistor[Resistor:R]: R, lcsc:R0402, F.Cu at (58.0, 67.0)
- added tester.pair2_rx2[1].indicator.led.led[LED:D]: D, lcsc:LED0805-R-RD, F.Cu at (62.0, 67.0)
- added tester.pair2_rx2[1].indicator.power_switch.mosfet[MOSFET:Q]: Q, lcsc:SOT-23-3_L2.9-W1.3-P1.90-LS2.4-BR, F.Cu at (54.0, 67.0)
- added tester.pair2_rx2[1].indicator.power_switch.pull_resistor[Resistor:R]: R, lcsc:R0402, F.Cu at (50.0, 67.0)
- added tester.pair3_tx1[0].indicator.led.current_limiting_resistor[Resistor:R]: R, lcsc:R0402, F.Cu at (58.0, 71.0)
- added tester.pair3_tx1[0].indicator.led.led[LED:D]: D, lcsc:LED0805-R-RD, F.Cu at (62.0, 71.0)
- added tester.pair3_tx1[0].indicator.power_switch.mosfet[MOSFET:Q]: Q, lcsc:SOT-23-3_L2.9-W1.3-P1.90-LS2.4-BR, F.Cu at (54.0, 71.0)
- added tester.pair3_tx1[0].indicator.power_switch.pull_resistor[Resistor:R]: R, lcsc:R0402, F.Cu at (50.0, 71.0)
- added tester.pair3_tx1[1].indicator.led.current_limiting_resistor[Resistor:R]: R, lcsc:R0402, F.Cu at (58.0, 75.0)
- added tester.pair3_tx1[1].indicator.led.led[LED:D]: D, lcsc:LED0805-R-RD, F.Cu at (62.0, 75.0)
- added tester.pair3_tx1[1].indicator.power_switch.mosfet[MOSFET:Q]: Q, lcsc:SOT-23-3_L2.9-W1.3-P1.90-LS2.4-BR, F.Cu at (54.0, 75.0)
- added tester.pair3_tx1[1].indicator.power_switch.pull_resistor[Resistor:R]: R, lcsc:R0402, F.Cu at (50.0, 75.0)
- added tester.pair4_tx2[0].indicator.led.current_limiting_resistor[Resistor:R]: R, lcsc:R0402, F.Cu at (58.0, 79.0)
- added tester.pair4_tx2[0].indicator.led.led[LED:D]: D, lcsc:LED0805-R-RD, F.Cu at (62.0, 79.0)
- added tester.pair4_tx2[0].indicator.power_switch.mosfet[MOSFET:Q]: Q, lcsc:SOT-23-3_L2.9-W1.3-P1.90-LS2.4-BR, F.Cu at (54.0, 79.0)
- added tester.pair4_tx2[0].indicator.power_switch.pull_resistor[Resistor:R]: R, lcsc:R0402, F.Cu at (50.0, 79.0)
- added tester.pair4_tx2[1].indicator.led.current_limiting_resistor[Resistor:R]: R, lcsc:R0402, F.Cu at (58.0, 83.0)
- added tester.pair4_tx2[1].indicator.led.led[LED:D]: D, lcsc:LED0805-R-RD, F.Cu at (62.0, 83.0)
- added tester.pair4_tx2[1].indicator.power_switch.mosfet[MOSFET:Q]: Q, lcsc:SOT-23-3_L2.9-W1.3-P1.90-LS2.4-BR, F.Cu at (54.0, 83.0)
- added tester.pair4_tx2[1].indicator.power_switch.pull_resistor[Resistor:R]: R, lcsc:R0402, F.Cu at (50.0, 83.0)
- added tester.rj45[0][RJ45_Receptacle:x]: x, lcsc:RJ45-TH_B-1-1, F.Cu at (141.7, 105.1)
- added tester.rj45[1][RJ45_Receptacle:x]: x, lcsc:RJ45-TH_B-1-1, F.Cu at (141.7, 122.3)
- added tester.sbu1.indicator.led.current_limiting_resistor[Resistor:R]: R, lcsc:R0402, F.Cu at (58.0, 87.0)
- added tester.sbu1.indicator.led.led[LED:D]: D, lcsc:LED0805-R-RD, F.Cu at (62.0, 87.0)
- added tester.sbu1.indicator.power_switch.mosfet[MOSFET:Q]: Q, lcsc:SOT-23-3_L2.9-W1.3-P1.90-LS2.4-BR, F.Cu at (54.0, 87.0)
- added tester.sbu1.indicator.power_switch.pull_resistor[Resistor:R]: R, lcsc:R0402, F.Cu at (50.0, 87.0)
- added tester.sbu2.indicator.led.current_limiting_resistor[Resistor:R]: R, lcsc:R0402, F.Cu at (58.0, 91.0)
- added tester.sbu2.indicator.led.led[LED:D]: D, lcsc:LED0805-R-RD, F.Cu at (62.0, 91.0)
- added tester.sbu2.indicator.power_switch.mosfet[MOSFET:Q]: Q, lcsc:SOT-23-3_L2.9-W1.3-P1.90-LS2.4-BR, F.Cu at (54.0, 91.0)
- added tester.sbu2.indicator.power_switch.pull_resistor[Resistor:R]: R, lcsc:R0402, F.Cu at (50.0, 91.0)
- added tester.shield.indicator.led.current_limiting_resistor[Resistor:R]: R, lcsc:R0402, F.Cu at (58.0, 95.0)
- added tester.shield.indicator.led.led[LED:D]: D, lcsc:LED0805-R-RD, F.Cu at (62.0, 95.0)
- added tester.shield.indicator.power_switch.mosfet[MOSFET:Q]: Q, lcsc:SOT-23-3_L2.9-W1.3-P1.90-LS2.4-BR, F.Cu at (54.0, 95.0)
- added tester.shield.indicator.power_switch.pull_resistor[Resistor:R]: R, lcsc:R0402, F.Cu at (50.0, 95.0)
- added tester.usb_c[0][USB_C_Receptacle:x]: x, lcsc:USB-C-SMD_TYPE-C-USB-18, F.Cu at (157.0, 104.1)
- added tester.usb_c[1][USB_C_Receptacle:x]: x, lcsc:USB-C-SMD_TYPE-C-USB-18, F.Cu at (157.0, 113.8)
- added tester.vbus[0].indicator.led.current_limiting_resistor[Resistor:R]: R, lcsc:R0402, F.Cu at (58.0, 99.0)
- added tester.vbus[0].indicator.led.led[LED:D]: D, lcsc:LED0805-R-RD, F.Cu at (62.0, 99.0)
- added tester.vbus[0].indicator.power_switch.mosfet[MOSFET:Q]: Q, lcsc:SOT-23-3_L2.9-W1.3-P1.90-LS2.4-BR, F.Cu at (54.0, 99.0)
- added tester.vbus[0].indicator.power_switch.pull_resistor[Resistor:R]: R, lcsc:R0402, F.Cu at (50.0, 99.0)
- added tester.vbus[1].indicator.led.current_limiting_resistor[Resistor:R]: R, lcsc:R0402, F.Cu at (58.0, 103.0)
- added tester.vbus[1].indicator.led.led[LED:D]: D, lcsc:LED0805-R-RD, F.Cu at (62.0, 103.0)
- added tester.vbus[1].indicator.power_switch.mosfet[MOSFET:Q]: Q, lcsc:SOT-23-3_L2.9-W1.3-P1.90-LS2.4-BR, F.Cu at (54.0, 103.0)
- added tester.vbus[1].indicator.power_switch.pull_resistor[Resistor:R]: R, lcsc:R0402, F.Cu at (50.0, 103.0)
- added tester.vbus[2].indicator.led.current_limiting_resistor[Resistor:R]: R, lcsc:R0402, F.Cu at (58.0, 107.0)
- added tester.vbus[2].indicator.led.led[LED:D]: D, lcsc:LED0805-R-RD, F.Cu at (62.0, 107.0)
- added tester.vbus[2].indicator.power_switch.mosfet[MOSFET:Q]: Q, lcsc:SOT-23-3_L2.9-W1.3-P1.90-LS2.4-BR, F.Cu at (54.0, 107.0)
- added tester.vbus[2].indicator.power_switch.pull_resistor[Resistor:R]: R, lcsc:R0402, F.Cu at (50.0, 107.0)
- added tester.vbus[3].indicator.led.current_limiting_resistor[Resistor:R]: R, lcsc:R0402, F.Cu at (58.0, 111.0)
- added tester.vbus[3].indicator.led.led[LED:D]: D, lcsc:LED0805-R-RD, F.Cu at (62.0, 111.0)
- added tester.vbus[3].indicator.power_switch.mosfet[MOSFET:Q]: Q, lcsc:SOT-23-3_L2.9-W1.3-P1.90-LS2.4-BR, F.Cu at (54.0, 111.0)
- added tester.vbus[3].indicator.power_switch.pull_resistor[Resistor:R]: R, lcsc:R0402, F.Cu at (50.0, 111.0)

Commit message: PCBTransformer & transformations
Parts:
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Connections:
- net psu.configuration_resistors[0][Resistor:5.0KΩ]-psu.usb[USB_C_Receptacle:x] renamed psu.usb[USB_C_Receptacle:x]-psu.configuration_resistors[0][Resistor:5.0KΩ]
- net tester.d1[0].indicator.led.led[LED:D]-tester.d1[0].indicator.led.current_limiting_resistor[Resistor:R] renamed tester.d1[0].indicator.led.current_limiting_resistor[Resistor:R]-tester.d1[0].indicator.led.led[LED:D]
- net tester.d1[1].indicator.led.led[LED:D]-tester.d1[1].indicator.led.current_limiting_resistor[Resistor:R] renamed tester.d1[1].indicator.led.current_limiting_resistor[Resistor:R]-tester.d1[1].indicator.led.led[LED:D]
- net tester.d2[0].indicator.led.current_limiting_resistor[Resistor:R]-tester.d2[0].indicator.led.led[LED:D] renamed tester.d2[0].indicator.led.led[LED:D]-tester.d2[0].indicator.led.current_limiting_resistor[Resistor:R]
- net tester.d2[1].indicator.power_switch[PowerSwitch:virt]:3-tester.d2[1].indicator.led[PoweredLED:virt]: renamed tester.d2[1].indicator.led[PoweredLED:virt]:2-tester.d2[1].indicator.power_switch[PowerSwitch:virt]:
- net tester.gnd[0].indicator.led.led[LED:D]-tester.gnd[0].indicator.led.current_limiting_resistor[Resistor:R] renamed tester.gnd[0].indicator.led.current_limiting_resistor[Resistor:R]-tester.gnd[0].indicator.led.led[LED:D]
- net tester.gnd[1].indicator.led.current_limiting_resistor[Resistor:R]-tester.gnd[1].indicator.led.led[LED:D] renamed tester.gnd[1].indicator.led.led[LED:D]-tester.gnd[1].indicator.led.current_limiting_resistor[Resistor:R]
- net tester.gnd[3].indicator.led.led[LED:D]-tester.gnd[3].indicator.led.current_limiting_resistor[Resistor:R] renamed tester.gnd[3].indicator.led.current_limiting_resistor[Resistor:R]-tester.gnd[3].indicator.led.led[LED:D]
- net tester.pair1_rx1[0].indicator.led.led[LED:D]-tester.pair1_rx1[0].indicator.led.current_limiting_resistor[Resistor:R] renamed tester.pair1_rx1[0].indicator.led.current_limiting_resistor[Resistor:R]-tester.pair1_rx1[0].indicator.led.led[LED:D]
- net tester.pair1_rx1[0].indicator.power_switch[PowerSwitch:virt]:3-tester.pair1_rx1[0].indicator.led[Pow renamed tester.pair1_rx1[0].indicator.led[PoweredLED:virt]:2-tester.pair1_rx1[0].indicator.power_switch[Powe
- net tester.pair1_rx1[1].indicator.led.current_limiting_resistor[Resistor:R]-tester.pair1_rx1[1].indicator.led.led[LED:D] renamed tester.pair1_rx1[1].indicator.led.led[LED:D]-tester.pair1_rx1[1].indicator.led.current_limiting_resistor[Resistor:R]
- net tester.pair2_rx2[0].indicator.led.current_limiting_resistor[Resistor:R]-tester.pair2_rx2[0].indicator.led.led[LED:D] renamed tester.pair2_rx2[0].indicator.led.led[LED:D]-tester.pair2_rx2[0].indicator.led.current_limiting_resistor[Resistor:R]
- net tester.pair2_rx2[0].indicator.led[PoweredLED:virt]:2-tester.pair2_rx2[0].indicator.power_switch[Powe renamed tester.pair2_rx2[0].indicator.power_switch[PowerSwitch:virt]:3-tester.pair2_rx2[0].indicator.led[Pow
- net tester.pair2_rx2[1].indicator.led.current_limiting_resistor[Resistor:R]-tester.pair2_rx2[1].indicator.led.led[LED:D] renamed tester.pair2_rx2[1].indicator.led.led[LED:D]-tester.pair2_rx2[1].indicator.led.current_limiting_resistor[Resistor:R]
- net tester.pair3_tx1[0].indicator.led.led[LED:D]-tester.pair3_tx1[0].indicator.led.current_limiting_resistor[Resistor:R] renamed tester.pair3_tx1[0].indicator.led.current_limiting_resistor[Resistor:R]-tester.pair3_tx1[0].indicator.led.led[LED:D]
- net tester.pair3_tx1[1].indicator.led.led[LED:D]-tester.pair3_tx1[1].indicator.led.current_limiting_resistor[Resistor:R] renamed tester.pair3_tx1[1].indicator.led.current_limiting_resistor[Resistor:R]-tester.pair3_tx1[1].indicator.led.led[LED:D]
- net tester.pair3_tx1[1].indicator.power_switch[PowerSwitch:virt]:3-tester.pair3_tx1[1].indicator.led[Pow renamed tester.pair3_tx1[1].indicator.led[PoweredLED:virt]:2-tester.pair3_tx1[1].indicator.power_switch[Powe
- net tester.pair4_tx2[1].indicator.power_switch[PowerSwitch:virt]:3-tester.pair4_tx2[1].indicator.led[Pow renamed tester.pair4_tx2[1].indicator.led[PoweredLED:virt]:2-tester.pair4_tx2[1].indicator.power_switch[Powe
- net tester.sbu1.indicator.led.led[LED:D]-tester.sbu1.indicator.led.current_limiting_resistor[Resistor:R] renamed tester.sbu1.indicator.led.current_limiting_resistor[Resistor:R]-tester.sbu1.indicator.led.led[LED:D]
- net tester.sbu2.indicator.led.current_limiting_resistor[Resistor:R]-tester.sbu2.indicator.led.led[LED:D] renamed tester.sbu2.indicator.led.led[LED:D]-tester.sbu2.indicator.led.current_limiting_resistor[Resistor:R]
- net tester.sbu2.indicator.led[PoweredLED:virt]:2-tester.sbu2.indicator.power_switch[PowerSwitch:virt]:3 renamed tester.sbu2.indicator.power_switch[PowerSwitch:virt]:3-tester.sbu2.indicator.led[PoweredLED:virt]:2
- net tester.shield.indicator.power_switch[PowerSwitch:virt]:2-tester.shield.indicator.led[PoweredLED:virt renamed tester.shield.indicator.led[PoweredLED:virt]-tester.shield.indicator.power_switch[PowerSwitch:virt]:
- net tester.vbus[0].indicator.led[PoweredLED:virt]:2-tester.vbus[0].indicator.power_switch[PowerSwitch:vi renamed tester.vbus[0].indicator.power_switch[PowerSwitch:virt]:3-tester.vbus[0].indicator.led[PoweredLED:vi
- net tester.vbus[1].indicator.led.current_limiting_resistor[Resistor:R]-tester.vbus[1].indicator.led.led[LED:D] renamed tester.vbus[1].indicator.led.led[LED:D]-tester.vbus[1].indicator.led.current_limiting_resistor[Resistor:R]
- net tester.vbus[1].indicator.led[PoweredLED:virt]:2-tester.vbus[1].indicator.power_switch[PowerSwitch:vi renamed tester.vbus[1].indicator.power_switch[PowerSwitch:virt]:3-tester.vbus[1].indicator.led[PoweredLED:vi
- net tester.vbus[2].indicator.led.led[LED:D]-tester.vbus[2].indicator.led.current_limiting_resistor[Resistor:R] renamed tester.vbus[2].indicator.led.current_limiting_resistor[Resistor:R]-tester.vbus[2].indicator.led.led[LED:D]
- net tester.vbus[2].indicator.led[PoweredLED:virt]:2-tester.vbus[2].indicator.power_switch[PowerSwitch:vi renamed tester.vbus[2].indicator.power_switch[PowerSwitch:virt]:3-tester.vbus[2].indicator.led[PoweredLED:vi
- net tester.vbus[3].indicator.led[PoweredLED:virt]:2-tester.vbus[3].indicator.power_switch[PowerSwitch:vi renamed tester.vbus[3].indicator.power_switch[PowerSwitch:virt]:3-tester.vbus[3].indicator.led[PoweredLED:vi
- psu.configuration_resistors[0][Resistor:5.0KΩ] pad 2: tester.pair1_rx1[0].indicator.power_switch[PowerSwitch:virt]:5-tester.gnd[3].indicator.power_switch[ -> tester.d2[1].indicator.power_switch[PowerSwitch:virt]:5-tester.gnd[1].indicator.power_switch[PowerSw
- psu.configuration_resistors[1][Resistor:5.0KΩ] pad 2: tester.pair1_rx1[0].indicator.power_switch[PowerSwitch:virt]:5-tester.gnd[3].indicator.power_switch[ -> tester.d2[1].indicator.power_switch[PowerSwitch:virt]:5-tester.gnd[1].indicator.power_switch[PowerSw
- psu.usb[USB_C_Receptacle:x] pad A1: tester.pair1_rx1[0].indicator.power_switch[PowerSwitch:virt]:5-tester.gnd[3].indicator.power_switch[ -> tester.d2[1].indicator.power_switch[PowerSwitch:virt]:5-tester.gnd[1].indicator.power_switch[PowerSw
- psu.usb[USB_C_Receptacle:x] pad A12: tester.pair1_rx1[0].indicator.power_switch[PowerSwitch:virt]:5-tester.gnd[3].indicator.power_switch[ -> tester.d2[1].indicator.power_switch[PowerSwitch:virt]:5-tester.gnd[1].indicator.power_switch[PowerSw
- psu.usb[USB_C_Receptacle:x] pad A4: tester.gnd[2].indicator.power_switch[PowerSwitch:virt]:4-tester.gnd[2][PairTester:virt]-tester.vbus[ -> tester.d1[1].indicator.power_switch[PowerSwitch:virt]:2-tester.pair4_tx2[0].indicator.led[PoweredLED
- psu.usb[USB_C_Receptacle:x] pad A9: tester.gnd[2].indicator.power_switch[PowerSwitch:virt]:4-tester.gnd[2][PairTester:virt]-tester.vbus[ -> tester.d1[1].indicator.power_switch[PowerSwitch:virt]:2-tester.pair4_tx2[0].indicator.led[PoweredLED
- psu.usb[USB_C_Receptacle:x] pad B1: tester.pair1_rx1[0].indicator.power_switch[PowerSwitch:virt]:5-tester.gnd[3].indicator.power_switch[ -> tester.d2[1].indicator.power_switch[PowerSwitch:virt]:5-tester.gnd[1].indicator.power_switch[PowerSw
- psu.usb[USB_C_Receptacle:x] pad B12: tester.pair1_rx1[0].indicator.power_switch[PowerSwitch:virt]:5-tester.gnd[3].indicator.power_switch[ -> tester.d2[1].indicator.power_switch[PowerSwitch:virt]:5-tester.gnd[1].indicator.power_switch[PowerSw
- psu.usb[USB_C_Receptacle:x] pad B4: tester.gnd[2].indicator.power_switch[PowerSwitch:virt]:4-tester.gnd[2][PairTester:virt]-tester.vbus[ -> tester.d1[1].indicator.power_switch[PowerSwitch:virt]:2-tester.pair4_tx2[0].indicator.led[PoweredLED
- psu.usb[USB_C_Receptacle:x] pad B9: tester.gnd[2].indicator.power_switch[PowerSwitch:virt]:4-tester.gnd[2][PairTester:virt]-tester.vbus[ -> tester.d1[1].indicator.power_switch[PowerSwitch:virt]:2-tester.pair4_tx2[0].indicator.led[PoweredLED
- tester.cc1.indicator.led.led[LED:D] pad 1: tester.gnd[2].indicator.power_switch[PowerSwitch:virt]:4-tester.gnd[2][PairTester:virt]-tester.vbus[ -> tester.d1[1].indicator.power_switch[PowerSwitch:virt]:2-tester.pair4_tx2[0].indicator.led[PoweredLED
- tester.cc1.indicator.power_switch.mosfet[MOSFET:Q] pad 1: tester.cc1.indicator.power_switch.pull_resistor[Resistor:R]-tester.cc1.indicator.power_switch.mosfet[MOSFET:Q] -> tester.cc1[PairTester:virt]:4-tester.cc1.indicator.power_switch[PowerSwitch:virt]-tester.cc1.indicat
- tester.cc1.indicator.power_switch.mosfet[MOSFET:Q] pad 3: tester.pair1_rx1[0].indicator.power_switch[PowerSwitch:virt]:5-tester.gnd[3].indicator.power_switch[ -> tester.d2[1].indicator.power_switch[PowerSwitch:virt]:5-tester.gnd[1].indicator.power_switch[PowerSw
- tester.cc1.indicator.power_switch.pull_resistor[Resistor:R] pad 1: tester.cc1.indicator.power_switch.pull_resistor[Resistor:R]-tester.cc1.indicator.power_switch.mosfet[MOSFET:Q] -> tester.cc1[PairTester:virt]:4-tester.cc1.indicator.power_switch[PowerSwitch:virt]-tester.cc1.indicat
- tester.cc2.indicator.led.led[LED:D] pad 1: tester.gnd[2].indicator.power_switch[PowerSwitch:virt]:4-tester.gnd[2][PairTester:virt]-tester.vbus[ -> tester.d1[1].indicator.power_switch[PowerSwitch:virt]:2-tester.pair4_tx2[0].indicator.led[PoweredLED
- tester.cc2.indicator.power_switch.mosfet[MOSFET:Q] pad 1: tester.cc2.indicator.power_switch.mosfet[MOSFET:Q]-tester.cc2.indicator.power_switch.pull_resistor[Resistor:R] -> tester.cc2.indicator[LEDIndicator:virt]-tester.cc2[PairTester:virt]:4-tester.cc2.indicator.power_swi
- tester.cc2.indicator.power_switch.mosfet[MOSFET:Q] pad 3: tester.pair1_rx1[0].indicator.power_switch[PowerSwitch:virt]:5-tester.gnd[3].indicator.power_switch[ -> tester.d2[1].indicator.power_switch[PowerSwitch:virt]:5-tester.gnd[1].indicator.power_switch[PowerSw
- tester.cc2.indicator.power_switch.pull_resistor[Resistor:R] pad 1: tester.cc2.indicator.power_switch.mosfet[MOSFET:Q]-tester.cc2.indicator.power_switch.pull_resistor[Resistor:R] -> tester.cc2.indicator[LEDIndicator:virt]-tester.cc2[PairTester:virt]:4-tester.cc2.indicator.power_swi
- tester.d1[0].indicator.led.led[LED:D] pad 1: tester.gnd[2].indicator.power_switch[PowerSwitch:virt]:4-tester.gnd[2][PairTester:virt]-tester.vbus[ -> tester.d1[1].indicator.power_switch[PowerSwitch:virt]:2-tester.pair4_tx2[0].indicator.led[PoweredLED
- tester.d1[0].indicator.power_switch.mosfet[MOSFET:Q] pad 1: tester.d1[0].indicator.power_switch.mosfet[MOSFET:Q]-tester.d1[0].indicator.power_switch.pull_resistor[Resistor:R] -> tester.d1[0].indicator.power_switch[PowerSwitch:virt]-tester.d1[0][PairTester:virt]:4-tester.d1[0].i
- tester.d1[0].indicator.power_switch.mosfet[MOSFET:Q] pad 3: tester.pair1_rx1[0].indicator.power_switch[PowerSwitch:virt]:5-tester.gnd[3].indicator.power_switch[ -> tester.d2[1].indicator.power_switch[PowerSwitch:virt]:5-tester.gnd[1].indicator.power_switch[PowerSw
- tester.d1[0].indicator.power_switch.pull_resistor[Resistor:R] pad 1: tester.d1[0].indicator.power_switch.mosfet[MOSFET:Q]-tester.d1[0].indicator.power_switch.pull_resistor[Resistor:R] -> tester.d1[0].indicator.power_switch[PowerSwitch:virt]-tester.d1[0][PairTester:virt]:4-tester.d1[0].i
- tester.d1[1].indicator.led.led[LED:D] pad 1: tester.gnd[2].indicator.power_switch[PowerSwitch:virt]:4-tester.gnd[2][PairTester:virt]-tester.vbus[ -> tester.d1[1].indicator.power_switch[PowerSwitch:virt]:2-tester.pair4_tx2[0].indicator.led[PoweredLED
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Routing:
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- added copper zone on F.Cu, net tester.d1[1].indicator.power_switch[PowerSwitch:virt]:2-tester.pair4_tx2[0].indicator.led[PoweredLED
Other:
- board outline added: 50 x 50 mm
- copper layers 2 -> 4

Commit message: Routing
Parts:
- moved psu.configuration_resistors[1][Resistor:5.0KΩ] 9.21 mm to (46.1, 39.7)
Routing:
- net tester.d2[1].indicator.power_switch[PowerSwitch:virt]:5-tester.gnd[1].indicator.power_switch[PowerSw: track 19.1 -> 217.6 mm, vias 1 -> 25
- net tester.d2[1][PairTester:virt]:4-tester.d2[1].indicator[LEDIndicator:virt]-tester.d2[1].indicator.pow: track 5.21 -> 66.7 mm, vias 2 -> 5
- net tester.shield.indicator[LEDIndicator:virt]-tester.shield[PairTester:virt]:4-tester.shield.indicator.: track 0.00 -> 60.0 mm, vias 1 -> 2
- net tester.pair2_rx2[1].indicator.power_switch[PowerSwitch:virt]-tester.pair2_rx2[1].indicator[LEDIndica: track 0.00 -> 57.7 mm, vias 1 -> 5
- net tester.pair4_tx2[1][PairTester:virt]:4-tester.pair4_tx2[1].indicator.power_switch[PowerSwitch:virt]-: track 3.79 -> 57.9 mm, vias 2 -> 6
- net tester.pair2_rx2[0].indicator[LEDIndicator:virt]-tester.pair2_rx2[0].indicator.power_switch[PowerSwi: track 0.00 -> 53.8 mm, vias 1 -> 3
- net tester.cc2.indicator[LEDIndicator:virt]-tester.cc2[PairTester:virt]:4-tester.cc2.indicator.power_swi: track 4.79 -> 54.6 mm, vias 2 -> 4
- net tester.d1[1].indicator.power_switch[PowerSwitch:virt]-tester.d1[1][PairTester:virt]:4-tester.d1[1].i: track 0.00 -> 47.9 mm, vias 1 -> 3
- net tester.sbu2[PairTester:virt]:4-tester.sbu2.indicator[LEDIndicator:virt]-tester.sbu2.indicator.power_: track 5.47 -> 53.1 mm, vias 2 -> 5
- net tester.pair3_tx1[1].indicator[LEDIndicator:virt]-tester.pair3_tx1[1].indicator.power_switch[PowerSwi: track 0.00 -> 45.8 mm, vias 1 -> 4
- net tester.d2[0].indicator.power_switch[PowerSwitch:virt]-tester.d2[0].indicator[LEDIndicator:virt]-test: track 4.70 -> 50.3 mm, vias 2 -> 5
- net tester.gnd[3][PairTester:virt]:4-tester.gnd[3].indicator[LEDIndicator:virt]-tester.gnd[3].indicator.: track 0.00 -> 44.7 mm, vias 1 -> 4
- net tester.pair3_tx1[0][PairTester:virt]:4-tester.pair3_tx1[0].indicator[LEDIndicator:virt]-tester.pair3: track 0.00 -> 44.1 mm, vias 1 -> 4
- net tester.pair1_rx1[1].indicator[LEDIndicator:virt]-tester.pair1_rx1[1].indicator.power_switch[PowerSwi: track 2.77 -> 45.7 mm
- net tester.pair4_tx2[0].indicator.power_switch[PowerSwitch:virt]-tester.pair4_tx2[0].indicator[LEDIndica: track 2.44 -> 44.7 mm, vias 2 -> 3
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
Commit message: Update requirements & Push dangling changes
Routing:
- net tester.vbus[3].indicator[LEDIndicator:virt]-tester.vbus[3].indicator.power_switch[PowerSwitch:virt]-: vias 4 -> 5
- net tester.vbus[2][PairTester:virt]:4-tester.vbus[2].indicator[LEDIndicator:virt]-tester.vbus[2].indicat: vias 3 -> 4
- net tester.vbus[1].indicator[LEDIndicator:virt]-tester.vbus[1][PairTester:virt]:4-tester.vbus[1].indicat: vias 3 -> 4
- net tester.vbus[0].indicator.power_switch[PowerSwitch:virt]-tester.vbus[0].indicator[LEDIndicator:virt]-: vias 3 -> 4
- net tester.shield.indicator[LEDIndicator:virt]-tester.shield[PairTester:virt]:4-tester.shield.indicator.: vias 2 -> 3
- net tester.sbu2[PairTester:virt]:4-tester.sbu2.indicator[LEDIndicator:virt]-tester.sbu2.indicator.power_: vias 5 -> 6
- net tester.sbu1.indicator[LEDIndicator:virt]-tester.sbu1[PairTester:virt]:4-tester.sbu1.indicator.power_: vias 3 -> 4
- net tester.pair4_tx2[1][PairTester:virt]:4-tester.pair4_tx2[1].indicator.power_switch[PowerSwitch:virt]-: vias 6 -> 7
- net tester.pair4_tx2[0].indicator.power_switch[PowerSwitch:virt]-tester.pair4_tx2[0].indicator[LEDIndica: vias 3 -> 4
- net tester.pair3_tx1[1].indicator[LEDIndicator:virt]-tester.pair3_tx1[1].indicator.power_switch[PowerSwi: vias 4 -> 5
- net tester.pair3_tx1[0][PairTester:virt]:4-tester.pair3_tx1[0].indicator[LEDIndicator:virt]-tester.pair3: vias 4 -> 5
- net tester.pair2_rx2[1].indicator.power_switch[PowerSwitch:virt]-tester.pair2_rx2[1].indicator[LEDIndica: vias 5 -> 6
- net tester.pair2_rx2[0].indicator[LEDIndicator:virt]-tester.pair2_rx2[0].indicator.power_switch[PowerSwi: vias 3 -> 4
- net tester.pair1_rx1[1].indicator[LEDIndicator:virt]-tester.pair1_rx1[1].indicator.power_switch[PowerSwi: vias 2 -> 3
- net tester.pair1_rx1[0][PairTester:virt]:4-tester.pair1_rx1[0].indicator[LEDIndicator:virt]-tester.pair1: vias 2 -> 3
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
Commit message: Finish routing & Fixing DRCs
Parts:
- added G***: Made with faebryk, logo:faebryk_logo, B.Cu at (22.9, 24.9)
- tester.cc1.indicator.led.current_limiting_resistor[Resistor:300Ω]: renamed from tester.cc1.indicator.led.current_limiting_resistor[Resistor:R]; value R -> 300Ω
- tester.cc1.indicator.power_switch.pull_resistor[Resistor:100KΩ]: renamed from tester.cc1.indicator.power_switch.pull_resistor[Resistor:R]; value R -> 100KΩ
- tester.cc2.indicator.led.current_limiting_resistor[Resistor:300Ω]: renamed from tester.cc2.indicator.led.current_limiting_resistor[Resistor:R]; value R -> 300Ω
- tester.cc2.indicator.power_switch.pull_resistor[Resistor:100KΩ]: renamed from tester.cc2.indicator.power_switch.pull_resistor[Resistor:R]; value R -> 100KΩ
- tester.d1[0].indicator.led.current_limiting_resistor[Resistor:300Ω]: renamed from tester.d1[0].indicator.led.current_limiting_resistor[Resistor:R]; value R -> 300Ω
- tester.d1[0].indicator.power_switch.pull_resistor[Resistor:100KΩ]: renamed from tester.d1[0].indicator.power_switch.pull_resistor[Resistor:R]; value R -> 100KΩ
- tester.d1[1].indicator.led.current_limiting_resistor[Resistor:300Ω]: renamed from tester.d1[1].indicator.led.current_limiting_resistor[Resistor:R]; value R -> 300Ω
- tester.d1[1].indicator.power_switch.pull_resistor[Resistor:100KΩ]: renamed from tester.d1[1].indicator.power_switch.pull_resistor[Resistor:R]; value R -> 100KΩ
- tester.d2[0].indicator.led.current_limiting_resistor[Resistor:300Ω]: renamed from tester.d2[0].indicator.led.current_limiting_resistor[Resistor:R]; value R -> 300Ω
- tester.d2[0].indicator.power_switch.pull_resistor[Resistor:100KΩ]: renamed from tester.d2[0].indicator.power_switch.pull_resistor[Resistor:R]; value R -> 100KΩ
- tester.d2[1].indicator.led.current_limiting_resistor[Resistor:300Ω]: renamed from tester.d2[1].indicator.led.current_limiting_resistor[Resistor:R]; value R -> 300Ω
- tester.d2[1].indicator.power_switch.pull_resistor[Resistor:100KΩ]: renamed from tester.d2[1].indicator.power_switch.pull_resistor[Resistor:R]; value R -> 100KΩ
- tester.gnd[0].indicator.led.current_limiting_resistor[Resistor:300Ω]: renamed from tester.gnd[0].indicator.led.current_limiting_resistor[Resistor:R]; value R -> 300Ω
- tester.gnd[0].indicator.power_switch.pull_resistor[Resistor:100KΩ]: renamed from tester.gnd[0].indicator.power_switch.pull_resistor[Resistor:R]; value R -> 100KΩ
- tester.gnd[1].indicator.led.current_limiting_resistor[Resistor:300Ω]: renamed from tester.gnd[1].indicator.led.current_limiting_resistor[Resistor:R]; value R -> 300Ω
- tester.gnd[1].indicator.power_switch.pull_resistor[Resistor:100KΩ]: renamed from tester.gnd[1].indicator.power_switch.pull_resistor[Resistor:R]; value R -> 100KΩ
- tester.gnd[2].indicator.led.current_limiting_resistor[Resistor:300Ω]: renamed from tester.gnd[2].indicator.led.current_limiting_resistor[Resistor:R]; value R -> 300Ω
- tester.gnd[2].indicator.power_switch.pull_resistor[Resistor:100KΩ]: renamed from tester.gnd[2].indicator.power_switch.pull_resistor[Resistor:R]; value R -> 100KΩ
- tester.gnd[3].indicator.led.current_limiting_resistor[Resistor:300Ω]: renamed from tester.gnd[3].indicator.led.current_limiting_resistor[Resistor:R]; value R -> 300Ω
- tester.gnd[3].indicator.power_switch.pull_resistor[Resistor:100KΩ]: renamed from tester.gnd[3].indicator.power_switch.pull_resistor[Resistor:R]; value R -> 100KΩ
- tester.pair1_rx1[0].indicator.led.current_limiting_resistor[Resistor:300Ω]: renamed from tester.pair1_rx1[0].indicator.led.current_limiting_resistor[Resistor:R]; value R -> 300Ω
- tester.pair1_rx1[0].indicator.power_switch.pull_resistor[Resistor:100KΩ]: renamed from tester.pair1_rx1[0].indicator.power_switch.pull_resistor[Resistor:R]; value R -> 100KΩ
- tester.pair1_rx1[1].indicator.led.current_limiting_resistor[Resistor:300Ω]: renamed from tester.pair1_rx1[1].indicator.led.current_limiting_resistor[Resistor:R]; value R -> 300Ω
- tester.pair1_rx1[1].indicator.power_switch.pull_resistor[Resistor:100KΩ]: renamed from tester.pair1_rx1[1].indicator.power_switch.pull_resistor[Resistor:R]; value R -> 100KΩ
- tester.pair2_rx2[0].indicator.led.current_limiting_resistor[Resistor:300Ω]: renamed from tester.pair2_rx2[0].indicator.led.current_limiting_resistor[Resistor:R]; value R -> 300Ω
- tester.pair2_rx2[0].indicator.power_switch.pull_resistor[Resistor:100KΩ]: renamed from tester.pair2_rx2[0].indicator.power_switch.pull_resistor[Resistor:R]; value R -> 100KΩ
- tester.pair2_rx2[1].indicator.led.current_limiting_resistor[Resistor:300Ω]: renamed from tester.pair2_rx2[1].indicator.led.current_limiting_resistor[Resistor:R]; value R -> 300Ω
- tester.pair2_rx2[1].indicator.power_switch.pull_resistor[Resistor:100KΩ]: renamed from tester.pair2_rx2[1].indicator.power_switch.pull_resistor[Resistor:R]; value R -> 100KΩ
- tester.pair3_tx1[0].indicator.led.current_limiting_resistor[Resistor:300Ω]: renamed from tester.pair3_tx1[0].indicator.led.current_limiting_resistor[Resistor:R]; value R -> 300Ω
- tester.pair3_tx1[0].indicator.power_switch.pull_resistor[Resistor:100KΩ]: renamed from tester.pair3_tx1[0].indicator.power_switch.pull_resistor[Resistor:R]; value R -> 100KΩ
- tester.pair3_tx1[1].indicator.led.current_limiting_resistor[Resistor:300Ω]: renamed from tester.pair3_tx1[1].indicator.led.current_limiting_resistor[Resistor:R]; value R -> 300Ω
- tester.pair3_tx1[1].indicator.power_switch.pull_resistor[Resistor:100KΩ]: renamed from tester.pair3_tx1[1].indicator.power_switch.pull_resistor[Resistor:R]; value R -> 100KΩ
- tester.pair4_tx2[0].indicator.led.current_limiting_resistor[Resistor:300Ω]: renamed from tester.pair4_tx2[0].indicator.led.current_limiting_resistor[Resistor:R]; value R -> 300Ω
- tester.pair4_tx2[0].indicator.power_switch.pull_resistor[Resistor:100KΩ]: renamed from tester.pair4_tx2[0].indicator.power_switch.pull_resistor[Resistor:R]; value R -> 100KΩ
- tester.pair4_tx2[1].indicator.led.current_limiting_resistor[Resistor:300Ω]: renamed from tester.pair4_tx2[1].indicator.led.current_limiting_resistor[Resistor:R]; value R -> 300Ω
- tester.pair4_tx2[1].indicator.power_switch.pull_resistor[Resistor:100KΩ]: renamed from tester.pair4_tx2[1].indicator.power_switch.pull_resistor[Resistor:R]; value R -> 100KΩ
- tester.sbu1.indicator.led.current_limiting_resistor[Resistor:300Ω]: renamed from tester.sbu1.indicator.led.current_limiting_resistor[Resistor:R]; value R -> 300Ω
- tester.sbu1.indicator.power_switch.pull_resistor[Resistor:100KΩ]: renamed from tester.sbu1.indicator.power_switch.pull_resistor[Resistor:R]; value R -> 100KΩ
- tester.sbu2.indicator.led.current_limiting_resistor[Resistor:300Ω]: renamed from tester.sbu2.indicator.led.current_limiting_resistor[Resistor:R]; value R -> 300Ω
- tester.sbu2.indicator.power_switch.pull_resistor[Resistor:100KΩ]: renamed from tester.sbu2.indicator.power_switch.pull_resistor[Resistor:R]; value R -> 100KΩ
- tester.shield.indicator.led.current_limiting_resistor[Resistor:300Ω]: renamed from tester.shield.indicator.led.current_limiting_resistor[Resistor:R]; value R -> 300Ω
- tester.shield.indicator.power_switch.pull_resistor[Resistor:100KΩ]: renamed from tester.shield.indicator.power_switch.pull_resistor[Resistor:R]; value R -> 100KΩ
- tester.vbus[0].indicator.led.current_limiting_resistor[Resistor:300Ω]: renamed from tester.vbus[0].indicator.led.current_limiting_resistor[Resistor:R]; value R -> 300Ω
- tester.vbus[0].indicator.power_switch.pull_resistor[Resistor:100KΩ]: renamed from tester.vbus[0].indicator.power_switch.pull_resistor[Resistor:R]; value R -> 100KΩ
- tester.vbus[1].indicator.led.current_limiting_resistor[Resistor:300Ω]: renamed from tester.vbus[1].indicator.led.current_limiting_resistor[Resistor:R]; value R -> 300Ω
- tester.vbus[1].indicator.power_switch.pull_resistor[Resistor:100KΩ]: renamed from tester.vbus[1].indicator.power_switch.pull_resistor[Resistor:R]; value R -> 100KΩ
- tester.vbus[2].indicator.led.current_limiting_resistor[Resistor:300Ω]: renamed from tester.vbus[2].indicator.led.current_limiting_resistor[Resistor:R]; value R -> 300Ω
- tester.vbus[2].indicator.power_switch.pull_resistor[Resistor:100KΩ]: renamed from tester.vbus[2].indicator.power_switch.pull_resistor[Resistor:R]; value R -> 100KΩ
- tester.vbus[3].indicator.led.current_limiting_resistor[Resistor:300Ω]: renamed from tester.vbus[3].indicator.led.current_limiting_resistor[Resistor:R]; value R -> 300Ω
- tester.vbus[3].indicator.power_switch.pull_resistor[Resistor:100KΩ]: renamed from tester.vbus[3].indicator.power_switch.pull_resistor[Resistor:R]; value R -> 100KΩ
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Connections:
- net psu.configuration_resistors[1][Resistor:5.0KΩ]-psu.usb[USB_C_Receptacle:x] renamed psu.usb[USB_C_Receptacle:x]-psu.configuration_resistors[1][Resistor:5.0KΩ]
- net psu.usb[USB_C_Receptacle:x]-psu.configuration_resistors[0][Resistor:5.0KΩ] renamed psu.configuration_resistors[0][Resistor:5.0KΩ]-psu.usb[USB_C_Receptacle:x]
- net tester.cc1.indicator.led.current_limiting_resistor[Resistor:R]-tester.cc1.indicator.led.led[LED:D] renamed tester.cc1.indicator.led.led[LED:D]-tester.cc1.indicator.led.current_limiting_resistor[Resistor:300Ω]
- net tester.cc1[PairTester:virt]:4-tester.cc1.indicator.power_switch[PowerSwitch:virt]-tester.cc1.indicat renamed tester.cc1[PairTester:virt]:4-tester.cc1.indicator[LEDIndicator:virt]-tester.cc1.indicator.power_swi
- net tester.cc2.indicator.led.led[LED:D]-tester.cc2.indicator.led.current_limiting_resistor[Resistor:R] renamed tester.cc2.indicator.led.current_limiting_resistor[Resistor:300Ω]-tester.cc2.indicator.led.led[LED:D]
- net tester.cc2.indicator.led[PoweredLED:virt]:2-tester.cc2.indicator.power_switch[PowerSwitch:virt]:3 renamed tester.cc2.indicator.power_switch[PowerSwitch:virt]:3-tester.cc2.indicator.led[PoweredLED:virt]:2
- net tester.cc2.indicator[LEDIndicator:virt]-tester.cc2[PairTester:virt]:4-tester.cc2.indicator.power_swi renamed tester.cc2[PairTester:virt]:4-tester.cc2.indicator.power_switch[PowerSwitch:virt]-tester.cc2.indicat
- net tester.d1[0].indicator.led.current_limiting_resistor[Resistor:R]-tester.d1[0].indicator.led.led[LED:D] renamed tester.d1[0].indicator.led.led[LED:D]-tester.d1[0].indicator.led.current_limiting_resistor[Resistor:300Ω]
- net tester.d1[1].indicator.led.current_limiting_resistor[Resistor:R]-tester.d1[1].indicator.led.led[LED:D] renamed tester.d1[1].indicator.led.current_limiting_resistor[Resistor:300Ω]-tester.d1[1].indicator.led.led[LED:D]
- net tester.d1[1].indicator.power_switch[PowerSwitch:virt]-tester.d1[1][PairTester:virt]:4-tester.d1[1].i renamed tester.d1[1].indicator.power_switch[PowerSwitch:virt]-tester.d1[1].indicator[LEDIndicator:virt]-test
- net tester.d1[1].indicator.power_switch[PowerSwitch:virt]:2-tester.pair4_tx2[0].indicator.led[PoweredLED renamed tester.d1[1].indicator.power_switch[PowerSwitch:virt]:4-tester.pair1_rx1[0].indicator.power_switch[P
- net tester.d2[0].indicator.led.led[LED:D]-tester.d2[0].indicator.led.current_limiting_resistor[Resistor:R] renamed tester.d2[0].indicator.led.current_limiting_resistor[Resistor:300Ω]-tester.d2[0].indicator.led.led[LED:D]
- net tester.d2[0].indicator.power_switch[PowerSwitch:virt]-tester.d2[0].indicator[LEDIndicator:virt]-test renamed tester.d2[0][PairTester:virt]:4-tester.d2[0].indicator.power_switch[PowerSwitch:virt]-tester.d2[0].i
- net tester.d2[1].indicator.led.led[LED:D]-tester.d2[1].indicator.led.current_limiting_resistor[Resistor:R] renamed tester.d2[1].indicator.led.current_limiting_resistor[Resistor:300Ω]-tester.d2[1].indicator.led.led[LED:D]
- net tester.d2[1].indicator.power_switch[PowerSwitch:virt]:5-tester.gnd[1].indicator.power_switch[PowerSw renamed tester.pair1_rx1[1][PairTester:virt]:2-tester.cc1[PairTester:virt]:2-tester.gnd[0].indicator.power_s
- net tester.d2[1][PairTester:virt]:4-tester.d2[1].indicator[LEDIndicator:virt]-tester.d2[1].indicator.pow renamed tester.d2[1].indicator.power_switch[PowerSwitch:virt]-tester.d2[1][PairTester:virt]:4-tester.d2[1].i
- net tester.gnd[0].indicator.led.current_limiting_resistor[Resistor:R]-tester.gnd[0].indicator.led.led[LED:D] renamed tester.gnd[0].indicator.led.led[LED:D]-tester.gnd[0].indicator.led.current_limiting_resistor[Resistor:300Ω]
- net tester.gnd[0].indicator.power_switch[PowerSwitch:virt]-tester.gnd[0][PairTester:virt]:4-tester.gnd[0 renamed tester.gnd[0].indicator[LEDIndicator:virt]-tester.gnd[0][PairTester:virt]:4-tester.gnd[0].indicator.
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Routing:
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Other:
- board text added: "USB-C CableTester v1.0.0 https://github.com/IoannisP-ITENG/CableTester"
