File: source/kicad/main/main.kicad_pcb (KiCad board)
At the start: 4 copper layers, 50 x 50 mm, 108 parts

Commit message: Place labels
Other:
- board text added: "cc1"
- board text added: "cc2"
- board text added: "d1[0]"
- board text added: "d1[1]"
- board text added: "d2[0]"
- board text added: "d2[1]"
- board text added: "gnd[0]"
- board text added: "gnd[1]"
- board text added: "gnd[2]"
- board text added: "gnd[3]"
- board text added: "pair1_rx1[0]"
- board text added: "pair1_rx1[1]"
- board text added: "pair2_rx2[0]"
- board text added: "pair2_rx2[1]"
- board text added: "pair3_tx1[0]"
- board text added: "pair3_tx1[1]"
- board text added: "pair4_tx2[0]"
- board text added: "pair4_tx2[1]"
- board text added: "sbu1"
- board text added: "sbu2"
- board text added: "shield"
- board text added: "vbus[0]"
- board text added: "vbus[1]"
- board text added: "vbus[2]"
- board text added: "vbus[3]"
- board text removed: "Shield"
Changed lines of the file:
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@@
       (stroke (width 0) (type solid)) (fill solid) (layer "B.SilkS"))
   )
-  (gr_line (start 50 0) (end 0 0)
-    (stroke (width 0.05) (type default)) (layer "Edge.Cuts"))
   (gr_line (start 0 0) (end 0 50)
     (stroke (width 0.05) (type default)) (layer "Edge.Cuts"))
   (gr_line (start 50 50) (end 50 0)
+    (stroke (width 0.05) (type default)) (layer "Edge.Cuts"))
+  (gr_line (start 50 0) (end 0 0)
     (stroke (width 0.05) (type default)) (layer "Edge.Cuts"))
   (gr_line (start 0 50) (end 50 50)
@@
     (effects (font (size 1 1) (thickness 0.15)) (justify left bottom mirror))
   )
-  (gr_text "Shield" (at 35.052 42.291 90) (layer "F.SilkS")
-    (effects (font (size 0.25 0.25) (thickness 0.0625)) (justify left bottom))
+  (gr_text "pair2_rx2[1]" (at 26 17.25) (layer "F.SilkS")
+    (effects (font (size 0.25 0.25) (thickness 0.0375)))
+  )
+  (gr_text "d2[0]" (at 21.25 10.75) (layer "F.SilkS")
+    (effects (font (size 0.25 0.25) (thickness 0.0375)))
+  )
+  (gr_text "d1[0]" (at 21.25 7.5) (layer "F.SilkS")
+    (effects (font (size 0.25 0.25) (thickness 0.0375)))
+  )
+  (gr_text "pair2_rx2[0]" (at 21.25 17.25) (layer "F.SilkS")
+    (effects (font (size 0.25 0.25) (thickness 0.0375)))
+  )
+  (gr_text "sbu2" (at 26 4.25) (layer "F.SilkS")
+    (effects (font (size 0.25 0.25) (thickness 0.0375)))
+  )
+  (gr_text "pair3_tx1[1]" (at 26 20.5) (layer "F.SilkS")
+    (effects (font (size 0.25 0.25) (thickness 0.0375)))
+  )
+  (gr_text "pair1_rx1[1]" (at 26 14) (layer "F.SilkS")
+    (effects (font (size 0.25 0.25) (thickness 0.0375)))
+  )
+  (gr_text "d2[1]" (at 26 10.75) (layer "F.SilkS")
+    (effects (font (size 0.25 0.25) (thickness 0.0375)))
+  )
+  (gr_text "gnd[1]" (at 27.25 30.25) (layer "F.SilkS")
+    (effects (font (size 0.25 0.25) (thickness 0.0375)))
+  )
+  (gr_text "vbus[1]" (at 21.25 30.25) (layer "F.SilkS")
+    (effects (font (size 0.25 0.25) (thickness 0.0375)))
+  )
+  (gr_text "pair3_tx1[0]" (at 21.25 20.5) (layer "F.SilkS")
+    (effects (font (size 0.25 0.25) (thickness 0.0375)))
+  )
+  (gr_text "gnd[0]" (at 27.25 27) (layer "F.SilkS")
+    (effects (font (size 0.25 0.25) (thickness 0.0375)))
+  )
+  (gr_text "pair4_tx2[0]" (at 21.25 23.75) (layer "F.SilkS")
+    (effects (font (size 0.25 0.25) (thickness 0.0375)))
+  )
+  (gr_text "vbus[2]" (at 21.25 33.5) (layer "F.SilkS")
+    (effects (font (size 0.25 0.25) (thickness 0.0375)))
+  )
+  (gr_text "vbus[0]" (at 21.25 27) (layer "F.SilkS")
+    (effects (font (size 0.25 0.25) (thickness 0.0375)))
+  )
+  (gr_text "sbu1" (at 21.25 4.25) (layer "F.SilkS")
+    (effects (font (size 0.25 0.25) (thickness 0.0375)))
+  )
+  (gr_text "cc2" (at 26 1) (layer "F.SilkS")
+    (effects (font (size 0.25 0.25) (thickness 0.0375)))
+  )
+  (gr_text "gnd[2]" (at 27.25 33.5) (layer "F.SilkS")
+    (effects (font (size 0.25 0.25) (thickness 0.0375)))
+  )
+  (gr_text "shield" (at 27.25 40) (layer "F.SilkS")
+    (effects (font (size 0.25 0.25) (thickness 0.0375)))
+  )
+  (gr_text "gnd[3]" (at 27.25 36.75) (layer "F.SilkS")
+    (effects (font (size 0.25 0.25) (thickness 0.0375)))
+  )
+  (gr_text "d1[1]" (at 26 7.5) (layer "F.SilkS")
+    (effects (font (size 0.25 0.25) (thickness 0.0375)))
+  )
+  (gr_text "cc1" (at 21.25 1) (layer "F.SilkS")
+    (effects (font (size 0.25 0.25) (thickness 0.0375)))
+  )
+  (gr_text "pair1_rx1[0]" (at 21.25 14) (layer "F.SilkS")
+    (effects (font (size 0.25 0.25) (thickness 0.0375)))
+  )
+  (gr_text "pair4_tx2[1]" (at 26 23.75) (layer "F.SilkS")
+    (effects (font (size 0.25 0.25) (thickness 0.0375)))
+  )
+  (gr_text "vbus[3]" (at 21.25 36.75) (layer "F.SilkS")
+    (effects (font (size 0.25 0.25) (thickness 0.0375)))
   )
   (segment (start 13.5 2.93) (end 14.48 2.93) (width 0.25) (layer "F.Cu") (net 1))
