File: src/kicad/main/main.kicad_pcb (KiCad board)
At the start: 4 copper layers, 50 x 50 mm, 108 parts

Commit message: Fix some leftover 2.0 migration problems
Parts:
- *.psu.configuration_resistors[0][Resistor:5.1kΩ]: renamed from psu.configuration_resistors[0][Resistor:5.0KΩ]; value 5.0KΩ -> 5.1kΩ
- *.psu.configuration_resistors[1][Resistor:5.1kΩ]: renamed from psu.configuration_resistors[1][Resistor:5.0KΩ]; value 5.0KΩ -> 5.1kΩ
- *.tester.cc1.indicator.led.current_limiting_resistor[Resistor:1.0kΩ]: renamed from tester.cc1.indicator.led.current_limiting_resistor[Resistor:1KΩ]; value 1KΩ -> 1.0kΩ
- *.tester.cc1.indicator.power_switch.pull_resistor[Resistor:100.0kΩ]: renamed from tester.cc1.indicator.power_switch.pull_resistor[Resistor:100KΩ]; value 100KΩ -> 100.0kΩ
- *.tester.cc2.indicator.led.current_limiting_resistor[Resistor:1.0kΩ]: renamed from tester.cc2.indicator.led.current_limiting_resistor[Resistor:1KΩ]; value 1KΩ -> 1.0kΩ
- *.tester.cc2.indicator.power_switch.pull_resistor[Resistor:100.0kΩ]: renamed from tester.cc2.indicator.power_switch.pull_resistor[Resistor:100KΩ]; value 100KΩ -> 100.0kΩ
- *.tester.d1[0].indicator.led.current_limiting_resistor[Resistor:1.0kΩ]: renamed from tester.d1[0].indicator.led.current_limiting_resistor[Resistor:1KΩ]; value 1KΩ -> 1.0kΩ
- *.tester.d1[0].indicator.power_switch.pull_resistor[Resistor:100.0kΩ]: renamed from tester.d1[0].indicator.power_switch.pull_resistor[Resistor:100KΩ]; value 100KΩ -> 100.0kΩ
- *.tester.d1[1].indicator.led.current_limiting_resistor[Resistor:1.0kΩ]: renamed from tester.d1[1].indicator.led.current_limiting_resistor[Resistor:1KΩ]; value 1KΩ -> 1.0kΩ
- *.tester.d1[1].indicator.power_switch.pull_resistor[Resistor:100.0kΩ]: renamed from tester.d1[1].indicator.power_switch.pull_resistor[Resistor:100KΩ]; value 100KΩ -> 100.0kΩ
- *.tester.d2[0].indicator.led.current_limiting_resistor[Resistor:1.0kΩ]: renamed from tester.d2[0].indicator.led.current_limiting_resistor[Resistor:1KΩ]; value 1KΩ -> 1.0kΩ
- *.tester.d2[0].indicator.power_switch.pull_resistor[Resistor:100.0kΩ]: renamed from tester.d2[0].indicator.power_switch.pull_resistor[Resistor:100KΩ]; value 100KΩ -> 100.0kΩ
- *.tester.d2[1].indicator.led.current_limiting_resistor[Resistor:1.0kΩ]: renamed from tester.d2[1].indicator.led.current_limiting_resistor[Resistor:1KΩ]; value 1KΩ -> 1.0kΩ
- *.tester.d2[1].indicator.power_switch.pull_resistor[Resistor:100.0kΩ]: renamed from tester.d2[1].indicator.power_switch.pull_resistor[Resistor:100KΩ]; value 100KΩ -> 100.0kΩ
- *.tester.gnd[0].indicator.led.current_limiting_resistor[Resistor:1.0kΩ]: renamed from tester.gnd[0].indicator.led.current_limiting_resistor[Resistor:1KΩ]; value 1KΩ -> 1.0kΩ
- *.tester.gnd[0].indicator.power_switch.pull_resistor[Resistor:100.0kΩ]: renamed from tester.gnd[0].indicator.power_switch.pull_resistor[Resistor:100KΩ]; value 100KΩ -> 100.0kΩ
- *.tester.gnd[1].indicator.led.current_limiting_resistor[Resistor:1.0kΩ]: renamed from tester.gnd[1].indicator.led.current_limiting_resistor[Resistor:1KΩ]; value 1KΩ -> 1.0kΩ
- *.tester.gnd[1].indicator.power_switch.pull_resistor[Resistor:100.0kΩ]: renamed from tester.gnd[1].indicator.power_switch.pull_resistor[Resistor:100KΩ]; value 100KΩ -> 100.0kΩ
- *.tester.gnd[2].indicator.led.current_limiting_resistor[Resistor:1.0kΩ]: renamed from tester.gnd[2].indicator.led.current_limiting_resistor[Resistor:1KΩ]; value 1KΩ -> 1.0kΩ
- *.tester.gnd[2].indicator.power_switch.pull_resistor[Resistor:100.0kΩ]: renamed from tester.gnd[2].indicator.power_switch.pull_resistor[Resistor:100KΩ]; value 100KΩ -> 100.0kΩ
- *.tester.gnd[3].indicator.led.current_limiting_resistor[Resistor:1.0kΩ]: renamed from tester.gnd[3].indicator.led.current_limiting_resistor[Resistor:1KΩ]; value 1KΩ -> 1.0kΩ
- *.tester.gnd[3].indicator.power_switch.pull_resistor[Resistor:100.0kΩ]: renamed from tester.gnd[3].indicator.power_switch.pull_resistor[Resistor:100KΩ]; value 100KΩ -> 100.0kΩ
- *.tester.pair1_rx1[0].indicator.led.current_limiting_resistor[Resistor:1.0kΩ]: renamed from tester.pair1_rx1[0].indicator.led.current_limiting_resistor[Resistor:1KΩ]; value 1KΩ -> 1.0kΩ
- *.tester.pair1_rx1[0].indicator.power_switch.pull_resistor[Resistor:100.0kΩ]: renamed from tester.pair1_rx1[0].indicator.power_switch.pull_resistor[Resistor:100KΩ]; value 100KΩ -> 100.0kΩ
- *.tester.pair1_rx1[1].indicator.led.current_limiting_resistor[Resistor:1.0kΩ]: renamed from tester.pair1_rx1[1].indicator.led.current_limiting_resistor[Resistor:1KΩ]; value 1KΩ -> 1.0kΩ
- *.tester.pair1_rx1[1].indicator.power_switch.pull_resistor[Resistor:100.0kΩ]: renamed from tester.pair1_rx1[1].indicator.power_switch.pull_resistor[Resistor:100KΩ]; value 100KΩ -> 100.0kΩ
- *.tester.pair2_rx2[0].indicator.led.current_limiting_resistor[Resistor:1.0kΩ]: renamed from tester.pair2_rx2[0].indicator.led.current_limiting_resistor[Resistor:1KΩ]; value 1KΩ -> 1.0kΩ
- *.tester.pair2_rx2[0].indicator.power_switch.pull_resistor[Resistor:100.0kΩ]: renamed from tester.pair2_rx2[0].indicator.power_switch.pull_resistor[Resistor:100KΩ]; value 100KΩ -> 100.0kΩ
- *.tester.pair2_rx2[1].indicator.led.current_limiting_resistor[Resistor:1.0kΩ]: renamed from tester.pair2_rx2[1].indicator.led.current_limiting_resistor[Resistor:1KΩ]; value 1KΩ -> 1.0kΩ
- *.tester.pair2_rx2[1].indicator.power_switch.pull_resistor[Resistor:100.0kΩ]: renamed from tester.pair2_rx2[1].indicator.power_switch.pull_resistor[Resistor:100KΩ]; value 100KΩ -> 100.0kΩ
- *.tester.pair3_tx1[0].indicator.led.current_limiting_resistor[Resistor:1.0kΩ]: renamed from tester.pair3_tx1[0].indicator.led.current_limiting_resistor[Resistor:1KΩ]; value 1KΩ -> 1.0kΩ
- *.tester.pair3_tx1[0].indicator.power_switch.pull_resistor[Resistor:100.0kΩ]: renamed from tester.pair3_tx1[0].indicator.power_switch.pull_resistor[Resistor:100KΩ]; value 100KΩ -> 100.0kΩ
- *.tester.pair3_tx1[1].indicator.led.current_limiting_resistor[Resistor:1.0kΩ]: renamed from tester.pair3_tx1[1].indicator.led.current_limiting_resistor[Resistor:1KΩ]; value 1KΩ -> 1.0kΩ
- *.tester.pair3_tx1[1].indicator.power_switch.pull_resistor[Resistor:100.0kΩ]: renamed from tester.pair3_tx1[1].indicator.power_switch.pull_resistor[Resistor:100KΩ]; value 100KΩ -> 100.0kΩ
- *.tester.pair4_tx2[0].indicator.led.current_limiting_resistor[Resistor:1.0kΩ]: renamed from tester.pair4_tx2[0].indicator.led.current_limiting_resistor[Resistor:1KΩ]; value 1KΩ -> 1.0kΩ
- *.tester.pair4_tx2[0].indicator.power_switch.pull_resistor[Resistor:100.0kΩ]: renamed from tester.pair4_tx2[0].indicator.power_switch.pull_resistor[Resistor:100KΩ]; value 100KΩ -> 100.0kΩ
- *.tester.pair4_tx2[1].indicator.led.current_limiting_resistor[Resistor:1.0kΩ]: renamed from tester.pair4_tx2[1].indicator.led.current_limiting_resistor[Resistor:1KΩ]; value 1KΩ -> 1.0kΩ
- *.tester.pair4_tx2[1].indicator.power_switch.pull_resistor[Resistor:100.0kΩ]: renamed from tester.pair4_tx2[1].indicator.power_switch.pull_resistor[Resistor:100KΩ]; value 100KΩ -> 100.0kΩ
- *.tester.sbu1.indicator.led.current_limiting_resistor[Resistor:1.0kΩ]: renamed from tester.sbu1.indicator.led.current_limiting_resistor[Resistor:1KΩ]; value 1KΩ -> 1.0kΩ
- *.tester.sbu1.indicator.power_switch.pull_resistor[Resistor:100.0kΩ]: renamed from tester.sbu1.indicator.power_switch.pull_resistor[Resistor:100KΩ]; value 100KΩ -> 100.0kΩ
- *.tester.sbu2.indicator.led.current_limiting_resistor[Resistor:1.0kΩ]: renamed from tester.sbu2.indicator.led.current_limiting_resistor[Resistor:1KΩ]; value 1KΩ -> 1.0kΩ
- *.tester.sbu2.indicator.power_switch.pull_resistor[Resistor:100.0kΩ]: renamed from tester.sbu2.indicator.power_switch.pull_resistor[Resistor:100KΩ]; value 100KΩ -> 100.0kΩ
- *.tester.shield.indicator.led.current_limiting_resistor[Resistor:1.0kΩ]: renamed from tester.shield.indicator.led.current_limiting_resistor[Resistor:1KΩ]; value 1KΩ -> 1.0kΩ
- *.tester.shield.indicator.power_switch.pull_resistor[Resistor:100.0kΩ]: renamed from tester.shield.indicator.power_switch.pull_resistor[Resistor:100KΩ]; value 100KΩ -> 100.0kΩ
- *.tester.vbus[0].indicator.led.current_limiting_resistor[Resistor:1.0kΩ]: renamed from tester.vbus[0].indicator.led.current_limiting_resistor[Resistor:1KΩ]; value 1KΩ -> 1.0kΩ
- *.tester.vbus[0].indicator.power_switch.pull_resistor[Resistor:100.0kΩ]: renamed from tester.vbus[0].indicator.power_switch.pull_resistor[Resistor:100KΩ]; value 100KΩ -> 100.0kΩ
- *.tester.vbus[1].indicator.led.current_limiting_resistor[Resistor:1.0kΩ]: renamed from tester.vbus[1].indicator.led.current_limiting_resistor[Resistor:1KΩ]; value 1KΩ -> 1.0kΩ
- *.tester.vbus[1].indicator.power_switch.pull_resistor[Resistor:100.0kΩ]: renamed from tester.vbus[1].indicator.power_switch.pull_resistor[Resistor:100KΩ]; value 100KΩ -> 100.0kΩ
- *.tester.vbus[2].indicator.led.current_limiting_resistor[Resistor:1.0kΩ]: renamed from tester.vbus[2].indicator.led.current_limiting_resistor[Resistor:1KΩ]; value 1KΩ -> 1.0kΩ
- *.tester.vbus[2].indicator.power_switch.pull_resistor[Resistor:100.0kΩ]: renamed from tester.vbus[2].indicator.power_switch.pull_resistor[Resistor:100KΩ]; value 100KΩ -> 100.0kΩ
- *.tester.vbus[3].indicator.led.current_limiting_resistor[Resistor:1.0kΩ]: renamed from tester.vbus[3].indicator.led.current_limiting_resistor[Resistor:1KΩ]; value 1KΩ -> 1.0kΩ
- *.tester.vbus[3].indicator.power_switch.pull_resistor[Resistor:100.0kΩ]: renamed from tester.vbus[3].indicator.power_switch.pull_resistor[Resistor:100KΩ]; value 100KΩ -> 100.0kΩ
- renumbered psu.usb[USB_C_Receptacle:x] to *.psu.usb[USB_Type_C_Receptacle_24_pin:x], tester.cc1.indicator.led.led[LED:D] to *.tester.cc1.indicator.led.led[LED:D], tester.cc1.indicator.power_switch.mosfet[MOSFET:Q] to *.tester.cc1.indicator.power_switch.mosfet[MOSFET:Q], tester.cc2.indicator.led.led[LED:D] to *.tester.cc2.indicator.led.led[LED:D], tester.cc2.indicator.power_switch.mosfet[MOSFET:Q] to *.tester.cc2.indicator.power_switch.mosfet[MOSFET:Q], tester.d1[0].indicator.led.led[LED:D] to *.tester.d1[0].indicator.led.led[LED:D], tester.d1[0].indicator.power_switch.mosfet[MOSFET:Q] to *.tester.d1[0].indicator.power_switch.mosfet[MOSFET:Q], tester.d1[1].indicator.led.led[LED:D] to *.tester.d1[1].indicator.led.led[LED:D], tester.d1[1].indicator.power_switch.mosfet[MOSFET:Q] to *.tester.d1[1].indicator.power_switch.mosfet[MOSFET:Q], tester.d2[0].indicator.led.led[LED:D] to *.tester.d2[0].indicator.led.led[LED:D], tester.d2[0].indicator.power_switch.mosfet[MOSFET:Q] to *.tester.d2[0].indicator.power_switch.mosfet[MOSFET:Q], tester.d2[1].indicator.led.led[LED:D] to *.tester.d2[1].indicator.led.led[LED:D], tester.d2[1].indicator.power_switch.mosfet[MOSFET:Q] to *.tester.d2[1].indicator.power_switch.mosfet[MOSFET:Q], tester.gnd[0].indicator.led.led[LED:D] to *.tester.gnd[0].indicator.led.led[LED:D], tester.gnd[0].indicator.power_switch.mosfet[MOSFET:Q] to *.tester.gnd[0].indicator.power_switch.mosfet[MOSFET:Q], tester.gnd[1].indicator.led.led[LED:D] to *.tester.gnd[1].indicator.led.led[LED:D], tester.gnd[1].indicator.power_switch.mosfet[MOSFET:Q] to *.tester.gnd[1].indicator.power_switch.mosfet[MOSFET:Q], tester.gnd[2].indicator.led.led[LED:D] to *.tester.gnd[2].indicator.led.led[LED:D], tester.gnd[2].indicator.power_switch.mosfet[MOSFET:Q] to *.tester.gnd[2].indicator.power_switch.mosfet[MOSFET:Q], tester.gnd[3].indicator.led.led[LED:D] to *.tester.gnd[3].indicator.led.led[LED:D], tester.gnd[3].indicator.power_switch.mosfet[MOSFET:Q] to *.tester.gnd[3].indicator.power_switch.mosfet[MOSFET:Q], tester.pair1_rx1[0].indicator.led.led[LED:D] to *.tester.pair1_rx1[0].indicator.led.led[LED:D], tester.pair1_rx1[0].indicator.power_switch.mosfet[MOSFET:Q] to *.tester.pair1_rx1[0].indicator.power_switch.mosfet[MOSFET:Q], tester.pair1_rx1[1].indicator.led.led[LED:D] to *.tester.pair1_rx1[1].indicator.led.led[LED:D], tester.pair1_rx1[1].indicator.power_switch.mosfet[MOSFET:Q] to *.tester.pair1_rx1[1].indicator.power_switch.mosfet[MOSFET:Q], tester.pair2_rx2[0].indicator.led.led[LED:D] to *.tester.pair2_rx2[0].indicator.led.led[LED:D], tester.pair2_rx2[0].indicator.power_switch.mosfet[MOSFET:Q] to *.tester.pair2_rx2[0].indicator.power_switch.mosfet[MOSFET:Q], tester.pair2_rx2[1].indicator.led.led[LED:D] to *.tester.pair2_rx2[1].indicator.led.led[LED:D], tester.pair2_rx2[1].indicator.power_switch.mosfet[MOSFET:Q] to *.tester.pair2_rx2[1].indicator.power_switch.mosfet[MOSFET:Q], tester.pair3_tx1[0].indicator.led.led[LED:D] to *.tester.pair3_tx1[0].indicator.led.led[LED:D], tester.pair3_tx1[0].indicator.power_switch.mosfet[MOSFET:Q] to *.tester.pair3_tx1[0].indicator.power_switch.mosfet[MOSFET:Q], tester.pair3_tx1[1].indicator.led.led[LED:D] to *.tester.pair3_tx1[1].indicator.led.led[LED:D], tester.pair3_tx1[1].indicator.power_switch.mosfet[MOSFET:Q] to *.tester.pair3_tx1[1].indicator.power_switch.mosfet[MOSFET:Q], tester.pair4_tx2[0].indicator.led.led[LED:D] to *.tester.pair4_tx2[0].indicator.led.led[LED:D], tester.pair4_tx2[0].indicator.power_switch.mosfet[MOSFET:Q] to *.tester.pair4_tx2[0].indicator.power_switch.mosfet[MOSFET:Q], tester.pair4_tx2[1].indicator.led.led[LED:D] to *.tester.pair4_tx2[1].indicator.led.led[LED:D], tester.pair4_tx2[1].indicator.power_switch.mosfet[MOSFET:Q] to *.tester.pair4_tx2[1].indicator.power_switch.mosfet[MOSFET:Q], tester.rj45[0][RJ45_Receptacle:x] to *.tester.rj45[0][RJ45_Receptacle:x], tester.rj45[1][RJ45_Receptacle:x] to *.tester.rj45[1][RJ45_Receptacle:x], tester.sbu1.indicator.led.led[LED:D] to *.tester.sbu1.indicator.led.led[LED:D], tester.sbu1.indicator.power_switch.mosfet[MOSFET:Q] to *.tester.sbu1.indicator.power_switch.mosfet[MOSFET:Q], tester.sbu2.indicator.led.led[LED:D] to *.tester.sbu2.indicator.led.led[LED:D], tester.sbu2.indicator.power_switch.mosfet[MOSFET:Q] to *.tester.sbu2.indicator.power_switch.mosfet[MOSFET:Q], tester.shield.indicator.led.led[LED:D] to *.tester.shield.indicator.led.led[LED:D], tester.shield.indicator.power_switch.mosfet[MOSFET:Q] to *.tester.shield.indicator.power_switch.mosfet[MOSFET:Q], tester.usb_c[0][USB_C_Receptacle:x] to *.tester.usb_c[0][USB_Type_C_Receptacle_24_pin:x], tester.usb_c[1][USB_C_Receptacle:x] to *.tester.usb_c[1][USB_Type_C_Receptacle_24_pin:x], tester.vbus[0].indicator.led.led[LED:D] to *.tester.vbus[0].indicator.led.led[LED:D], tester.vbus[0].indicator.power_switch.mosfet[MOSFET:Q] to *.tester.vbus[0].indicator.power_switch.mosfet[MOSFET:Q], tester.vbus[1].indicator.led.led[LED:D] to *.tester.vbus[1].indicator.led.led[LED:D], tester.vbus[1].indicator.power_switch.mosfet[MOSFET:Q] to *.tester.vbus[1].indicator.power_switch.mosfet[MOSFET:Q], tester.vbus[2].indicator.led.led[LED:D] to *.tester.vbus[2].indicator.led.led[LED:D], tester.vbus[2].indicator.power_switch.mosfet[MOSFET:Q] to *.tester.vbus[2].indicator.power_switch.mosfet[MOSFET:Q], tester.vbus[3].indicator.led.led[LED:D] to *.tester.vbus[3].indicator.led.led[LED:D], tester.vbus[3].indicator.power_switch.mosfet[MOSFET:Q] to *.tester.vbus[3].indicator.power_switch.mosfet[MOSFET:Q]
Connections:
- net psu.usb[USB_C_Receptacle:x]-psu.configuration_resistors[0][Resistor:5.0KΩ] renamed *.psu.usb[USB_Type_C_Receptacle_24_pin:x]-psu.configuration_resistors[0][Resistor:5.1kΩ]
- net psu.usb[USB_C_Receptacle:x]-psu.configuration_resistors[1][Resistor:5.0KΩ] renamed *.psu.usb[USB_Type_C_Receptacle_24_pin:x]-psu.configuration_resistors[1][Resistor:5.1kΩ]
- net tester.cc1.indicator.led.current_limiting_resistor[Resistor:1KΩ]-tester.cc1.indicator.led.led[LED:D] renamed *.tester.cc1.indicator.led.current_limiting_resistor[Resistor:1.0kΩ]-*.tester.cc1.indicator.led.led[LED:D]
- net tester.cc1.indicator.power_switch[PowerSwitch:virt]:5-tester.cc1.indicator.led[PoweredLED:virt]:2 renamed *.tester.cc1.indicator.power_switch[PowerSwitch:virt]:5-*.tester.cc1.indicator.led[PoweredLED:virt]:2
- net tester.cc1.indicator[LEDIndicator:virt]-tester.cc1.indicator.power_switch[PowerSwitch:virt]-tester.c renamed *.tester.cc1.indicator[LEDIndicator:virt]-*.tester.cc1.indicator.power_switch[PowerSwitch:virt]-*.tester.c
- net tester.cc2.indicator.led.led[LED:D]-tester.cc2.indicator.led.current_limiting_resistor[Resistor:1KΩ] renamed *.tester.cc2.indicator.led.led[LED:D]-*.tester.cc2.indicator.led.current_limiting_resistor[Resistor:1.0kΩ]
- net tester.cc2.indicator.power_switch[PowerSwitch:virt]-tester.cc2.indicator[LEDIndicator:virt]-tester.c renamed *.tester.cc2.indicator.power_switch[PowerSwitch:virt]-*.tester.cc2.indicator[LEDIndicator:virt]-*.tester.c
- net tester.cc2.indicator.power_switch[PowerSwitch:virt]:5-tester.cc2.indicator.led[PoweredLED:virt]:2 renamed *.tester.cc2.indicator.power_switch[PowerSwitch:virt]:5-*.tester.cc2.indicator.led[PoweredLED:virt]:2
- net tester.d1[0].indicator.led.current_limiting_resistor[Resistor:1KΩ]-tester.d1[0].indicator.led.led[LED:D] renamed *.tester.d1[0].indicator.led.current_limiting_resistor[Resistor:1.0kΩ]-*.tester.d1[0].indicator.led.led[LED:D]
- net tester.d1[0].indicator.led[PoweredLED:virt]:2-tester.d1[0].indicator.power_switch[PowerSwitch:virt]: renamed *.tester.d1[0].indicator.led[PoweredLED:virt]:2-*.tester.d1[0].indicator.power_switch[PowerSwitch:virt]:
- net tester.d1[0].indicator[LEDIndicator:virt]-tester.d1[0].indicator.power_switch[PowerSwitch:virt]-test renamed *.tester.d1[0].indicator[LEDIndicator:virt]-*.tester.d1[0].indicator.power_switch[PowerSwitch:virt]-test
- net tester.d1[1].indicator.led.led[LED:D]-tester.d1[1].indicator.led.current_limiting_resistor[Resistor:1KΩ] renamed *.tester.d1[1].indicator.led.led[LED:D]-*.tester.d1[1].indicator.led.current_limiting_resistor[Resistor:1.0kΩ]
- net tester.d1[1].indicator.power_switch[PowerSwitch:virt]-tester.d1[1][PairTester:virt]:4-tester.d1[1].i renamed *.tester.d1[1].indicator.power_switch[PowerSwitch:virt]-*.tester.d1[1][Pair*.tester:virt]:4-*.tester.d1[1].i
- net tester.d1[1].indicator.power_switch[PowerSwitch:virt]:5-tester.d1[1].indicator.led[PoweredLED:virt]: renamed *.tester.d1[1].indicator.power_switch[PowerSwitch:virt]:5-*.tester.d1[1].indicator.led[PoweredLED:virt]:
- net tester.d2[0].indicator.led.current_limiting_resistor[Resistor:1KΩ]-tester.d2[0].indicator.led.led[LED:D] renamed *.tester.d2[0].indicator.led.current_limiting_resistor[Resistor:1.0kΩ]-*.tester.d2[0].indicator.led.led[LED:D]
- net tester.d2[0].indicator.power_switch[PowerSwitch:virt]:5-tester.d2[0].indicator.led[PoweredLED:virt]: renamed *.tester.d2[0].indicator.power_switch[PowerSwitch:virt]:5-*.tester.d2[0].indicator.led[PoweredLED:virt]:
- net tester.d2[0][PairTester:virt]:4-tester.d2[0].indicator.power_switch[PowerSwitch:virt]-tester.d2[0].i renamed *.tester.d2[0][Pair*.tester:virt]:4-*.tester.d2[0].indicator.power_switch[PowerSwitch:virt]-*.tester.d2[0].i
- net tester.d2[1].indicator.led.current_limiting_resistor[Resistor:1KΩ]-tester.d2[1].indicator.led.led[LED:D] renamed *.tester.d2[1].indicator.led.current_limiting_resistor[Resistor:1.0kΩ]-*.tester.d2[1].indicator.led.led[LED:D]
- net tester.d2[1].indicator.power_switch[PowerSwitch:virt]:5-tester.d2[1].indicator.led[PoweredLED:virt]: renamed *.tester.d2[1].indicator.power_switch[PowerSwitch:virt]:5-*.tester.d2[1].indicator.led[PoweredLED:virt]:
- net tester.d2[1][PairTester:virt]:4-tester.d2[1].indicator[LEDIndicator:virt]-tester.d2[1].indicator.pow renamed *.tester.d2[1][Pair*.tester:virt]:4-*.tester.d2[1].indicator[LEDIndicator:virt]-*.tester.d2[1].indicator.pow
- net tester.gnd[0].indicator.led.led[LED:D]-tester.gnd[0].indicator.led.current_limiting_resistor[Resistor:1KΩ] renamed *.tester.gnd[0].indicator.led.led[LED:D]-*.tester.gnd[0].indicator.led.current_limiting_resistor[Resistor:1.0kΩ]
- net tester.gnd[0].indicator.power_switch[PowerSwitch:virt]-tester.gnd[0].indicator[LEDIndicator:virt]-te renamed *.tester.gnd[0].indicator.power_switch[PowerSwitch:virt]-*.tester.gnd[0].indicator[LEDIndicator:virt]-te
- net tester.gnd[0].indicator.power_switch[PowerSwitch:virt]:4-tester.gnd[0].indicator.led[PoweredLED:virt renamed *.tester.gnd[0].indicator.power_switch[PowerSwitch:virt]:4-*.tester.gnd[0].indicator.led[PoweredLED:virt
- net tester.gnd[1].indicator.led.led[LED:D]-tester.gnd[1].indicator.led.current_limiting_resistor[Resistor:1KΩ] renamed *.tester.gnd[1].indicator.led.led[LED:D]-*.tester.gnd[1].indicator.led.current_limiting_resistor[Resistor:1.0kΩ]
- net tester.gnd[1].indicator.power_switch[PowerSwitch:virt]:4-tester.gnd[1].indicator.led[PoweredLED:virt renamed *.tester.gnd[1].indicator.power_switch[PowerSwitch:virt]:4-*.tester.gnd[1].indicator.led[PoweredLED:virt
- net tester.gnd[1][PairTester:virt]:4-tester.gnd[1].indicator.power_switch[PowerSwitch:virt]-tester.gnd[1 renamed *.tester.gnd[1][Pair*.tester:virt]:4-*.tester.gnd[1].indicator.power_switch[PowerSwitch:virt]-*.tester.gnd[1
- net tester.gnd[2].indicator.led.led[LED:D]-tester.gnd[2].indicator.led.current_limiting_resistor[Resistor:1KΩ] renamed *.tester.gnd[2].indicator.led.led[LED:D]-*.tester.gnd[2].indicator.led.current_limiting_resistor[Resistor:1.0kΩ]
- net tester.gnd[2].indicator.led[PoweredLED:virt]-tester.gnd[2].indicator.power_switch[PowerSwitch:virt]: renamed *.tester.gnd[2].indicator.led[PoweredLED:virt]-*.tester.gnd[2].indicator.power_switch[PowerSwitch:virt]:
- net tester.gnd[2][PairTester:virt]:4-tester.gnd[2].indicator[LEDIndicator:virt]-tester.gnd[2].indicator. renamed *.tester.gnd[2][Pair*.tester:virt]:4-*.tester.gnd[2].indicator[LEDIndicator:virt]-*.tester.gnd[2].indicator.
- net tester.gnd[3].indicator.led.led[LED:D]-tester.gnd[3].indicator.led.current_limiting_resistor[Resistor:1KΩ] renamed *.tester.gnd[3].indicator.led.led[LED:D]-*.tester.gnd[3].indicator.led.current_limiting_resistor[Resistor:1.0kΩ]
- net tester.gnd[3].indicator.led[PoweredLED:virt]-tester.gnd[3].indicator.power_switch[PowerSwitch:virt]: renamed *.tester.gnd[3].indicator.led[PoweredLED:virt]-*.tester.gnd[3].indicator.power_switch[PowerSwitch:virt]:
- net tester.gnd[3][PairTester:virt]:4-tester.gnd[3].indicator[LEDIndicator:virt]-tester.gnd[3].indicator. renamed *.tester.gnd[3][Pair*.tester:virt]:4-*.tester.gnd[3].indicator[LEDIndicator:virt]-*.tester.gnd[3].indicator.
- net tester.pair1_rx1[0].indicator.led.led[LED:D]-tester.pair1_rx1[0].indicator.led.current_limiting_resistor[Resistor:1KΩ] renamed *.tester.pair1_rx1[0].indicator.led.led[LED:D]-*.tester.pair1_rx1[0].indicator.led.current_limiting_resistor[Resistor:1.0kΩ]
- net tester.pair1_rx1[0].indicator.led[PoweredLED:virt]:2-tester.pair1_rx1[0].indicator.power_switch[Powe renamed *.tester.pair1_rx1[0].indicator.led[PoweredLED:virt]:2-*.tester.pair1_rx1[0].indicator.power_switch[Powe
- net tester.pair1_rx1[0][PairTester:virt]:4-tester.pair1_rx1[0].indicator.power_switch[PowerSwitch:virt]- renamed *.tester.pair1_rx1[0][Pair*.tester:virt]:4-*.tester.pair1_rx1[0].indicator.power_switch[PowerSwitch:virt]-
- net tester.pair1_rx1[1].indicator.led.current_limiting_resistor[Resistor:1KΩ]-tester.pair1_rx1[1].indicator.led.led[LED:D] renamed *.tester.pair1_rx1[1].indicator.led.current_limiting_resistor[Resistor:1.0kΩ]-*.tester.pair1_rx1[1].indicator.led.led[LED:D]
- net tester.pair1_rx1[1].indicator.led[PoweredLED:virt]-tester.d2[1].indicator.power_switch[PowerSwitch:v renamed *.tester.pair1_rx1[1].indicator.led[PoweredLED:virt]-*.tester.d2[1].indicator.power_switch[PowerSwitch:v
- net tester.pair1_rx1[1].indicator.power_switch[PowerSwitch:virt]:5-tester.pair1_rx1[1].indicator.led[Pow renamed *.tester.pair1_rx1[1].indicator.power_switch[PowerSwitch:virt]:5-*.tester.pair1_rx1[1].indicator.led[Pow
- net tester.pair1_rx1[1][PairTester:virt]:4-tester.pair1_rx1[1].indicator[LEDIndicator:virt]-tester.pair1 renamed *.tester.pair1_rx1[1][Pair*.tester:virt]:4-*.tester.pair1_rx1[1].indicator[LEDIndicator:virt]-*.tester.pair1
- net tester.pair2_rx2[0].indicator.led.led[LED:D]-tester.pair2_rx2[0].indicator.led.current_limiting_resistor[Resistor:1KΩ] renamed *.tester.pair2_rx2[0].indicator.led.led[LED:D]-*.tester.pair2_rx2[0].indicator.led.current_limiting_resistor[Resistor:1.0kΩ]
- net tester.pair2_rx2[0].indicator.power_switch[PowerSwitch:virt]:5-tester.pair2_rx2[0].indicator.led[Pow renamed *.tester.pair2_rx2[0].indicator.power_switch[PowerSwitch:virt]:5-*.tester.pair2_rx2[0].indicator.led[Pow
- net tester.pair2_rx2[0].indicator[LEDIndicator:virt]-tester.pair2_rx2[0][PairTester:virt]:4-tester.pair2 renamed *.tester.pair2_rx2[0].indicator[LEDIndicator:virt]-*.tester.pair2_rx2[0][Pair*.tester:virt]:4-*.tester.pair2
- net tester.pair2_rx2[1].indicator.led.current_limiting_resistor[Resistor:1KΩ]-tester.pair2_rx2[1].indicator.led.led[LED:D] renamed *.tester.pair2_rx2[1].indicator.led.current_limiting_resistor[Resistor:1.0kΩ]-*.tester.pair2_rx2[1].indicator.led.led[LED:D]
- net tester.pair2_rx2[1].indicator.power_switch[PowerSwitch:virt]-tester.pair2_rx2[1].indicator[LEDIndica renamed *.tester.pair2_rx2[1].indicator.power_switch[PowerSwitch:virt]-*.tester.pair2_rx2[1].indicator[LEDIndica
- net tester.pair2_rx2[1].indicator.power_switch[PowerSwitch:virt]:5-tester.pair2_rx2[1].indicator.led[Pow renamed *.tester.pair2_rx2[1].indicator.power_switch[PowerSwitch:virt]:5-*.tester.pair2_rx2[1].indicator.led[Pow
- net tester.pair3_tx1[0].indicator.led.current_limiting_resistor[Resistor:1KΩ]-tester.pair3_tx1[0].indicator.led.led[LED:D] renamed *.tester.pair3_tx1[0].indicator.led.current_limiting_resistor[Resistor:1.0kΩ]-*.tester.pair3_tx1[0].indicator.led.led[LED:D]
- net tester.pair3_tx1[0].indicator.power_switch[PowerSwitch:virt]-tester.pair3_tx1[0][PairTester:virt]:4- renamed *.tester.pair3_tx1[0].indicator.power_switch[PowerSwitch:virt]-*.tester.pair3_tx1[0][Pair*.tester:virt]:4-
- net tester.pair3_tx1[0].indicator.power_switch[PowerSwitch:virt]:5-tester.pair3_tx1[0].indicator.led[Pow renamed *.tester.pair3_tx1[0].indicator.power_switch[PowerSwitch:virt]:5-*.tester.pair3_tx1[0].indicator.led[Pow
- net tester.pair3_tx1[1].indicator.led.current_limiting_resistor[Resistor:1KΩ]-tester.pair3_tx1[1].indicator.led.led[LED:D] renamed *.tester.pair3_tx1[1].indicator.led.current_limiting_resistor[Resistor:1.0kΩ]-*.tester.pair3_tx1[1].indicator.led.led[LED:D]
- net tester.pair3_tx1[1].indicator.power_switch[PowerSwitch:virt]:5-tester.pair3_tx1[1].indicator.led[Pow renamed *.tester.pair3_tx1[1].indicator.power_switch[PowerSwitch:virt]:5-*.tester.pair3_tx1[1].indicator.led[Pow
- net tester.pair3_tx1[1].indicator[LEDIndicator:virt]-tester.pair3_tx1[1][PairTester:virt]:4-tester.pair3 renamed *.tester.pair3_tx1[1].indicator[LEDIndicator:virt]-*.tester.pair3_tx1[1][Pair*.tester:virt]:4-*.tester.pair3
- net tester.pair4_tx2[0].indicator.led.led[LED:D]-tester.pair4_tx2[0].indicator.led.current_limiting_resistor[Resistor:1KΩ] renamed *.tester.pair4_tx2[0].indicator.led.led[LED:D]-*.tester.pair4_tx2[0].indicator.led.current_limiting_resistor[Resistor:1.0kΩ]
- net tester.pair4_tx2[0].indicator.power_switch[PowerSwitch:virt]:5-tester.pair4_tx2[0].indicator.led[Pow renamed *.tester.pair4_tx2[0].indicator.power_switch[PowerSwitch:virt]:5-*.tester.pair4_tx2[0].indicator.led[Pow
- net tester.pair4_tx2[0].indicator[LEDIndicator:virt]-tester.pair4_tx2[0].indicator.power_switch[PowerSwi renamed *.tester.pair4_tx2[0].indicator[LEDIndicator:virt]-*.tester.pair4_tx2[0].indicator.power_switch[PowerSwi
- net tester.pair4_tx2[1].indicator.led.led[LED:D]-tester.pair4_tx2[1].indicator.led.current_limiting_resistor[Resistor:1KΩ] renamed *.tester.pair4_tx2[1].indicator.led.led[LED:D]-*.tester.pair4_tx2[1].indicator.led.current_limiting_resistor[Resistor:1.0kΩ]
- net tester.pair4_tx2[1].indicator.power_switch[PowerSwitch:virt]:5-tester.pair4_tx2[1].indicator.led[Pow renamed *.tester.pair4_tx2[1].indicator.power_switch[PowerSwitch:virt]:5-*.tester.pair4_tx2[1].indicator.led[Pow
- net tester.pair4_tx2[1].indicator[LEDIndicator:virt]-tester.pair4_tx2[1].indicator.power_switch[PowerSwi renamed *.tester.pair4_tx2[1].indicator[LEDIndicator:virt]-*.tester.pair4_tx2[1].indicator.power_switch[PowerSwi
- net tester.sbu1.indicator.led.led[LED:D]-tester.sbu1.indicator.led.current_limiting_resistor[Resistor:1KΩ] renamed *.tester.sbu1.indicator.led.led[LED:D]-*.tester.sbu1.indicator.led.current_limiting_resistor[Resistor:1.0kΩ]
- net tester.sbu1.indicator.led[PoweredLED:virt]:2-tester.sbu1.indicator.power_switch[PowerSwitch:virt]:5 renamed *.tester.sbu1.indicator.led[PoweredLED:virt]:2-*.tester.sbu1.indicator.power_switch[PowerSwitch:virt]:5
- net tester.sbu1.indicator[LEDIndicator:virt]-tester.sbu1.indicator.power_switch[PowerSwitch:virt]-tester renamed *.tester.sbu1.indicator[LEDIndicator:virt]-*.tester.sbu1.indicator.power_switch[PowerSwitch:virt]-*.tester
- net tester.sbu2.indicator.led.led[LED:D]-tester.sbu2.indicator.led.current_limiting_resistor[Resistor:1KΩ] renamed *.tester.sbu2.indicator.led.led[LED:D]-*.tester.sbu2.indicator.led.current_limiting_resistor[Resistor:1.0kΩ]
- net tester.sbu2.indicator.power_switch[PowerSwitch:virt]-tester.sbu2[PairTester:virt]:4-tester.sbu2.indi renamed *.tester.sbu2.indicator.power_switch[PowerSwitch:virt]-*.tester.sbu2[Pair*.tester:virt]:4-*.tester.sbu2.indi
- net tester.sbu2.indicator.power_switch[PowerSwitch:virt]:5-tester.sbu2.indicator.led[PoweredLED:virt]:2 renamed *.tester.sbu2.indicator.power_switch[PowerSwitch:virt]:5-*.tester.sbu2.indicator.led[PoweredLED:virt]:2
- net tester.shield.indicator.led.led[LED:D]-tester.shield.indicator.led.current_limiting_resistor[Resistor:1KΩ] renamed *.tester.shield.indicator.led.led[LED:D]-*.tester.shield.indicator.led.current_limiting_resistor[Resistor:1.0kΩ]
- net tester.shield.indicator.led[PoweredLED:virt]-tester.shield.indicator.power_switch[PowerSwitch:virt]: renamed *.tester.shield.indicator.led[PoweredLED:virt]-*.tester.shield.indicator.power_switch[PowerSwitch:virt]:
- net tester.shield.indicator.power_switch[PowerSwitch:virt]-tester.shield.indicator[LEDIndicator:virt]-te renamed *.tester.shield.indicator.power_switch[PowerSwitch:virt]-*.tester.shield.indicator[LEDIndicator:virt]-te
- net tester.vbus[0].indicator.led.led[LED:D]-tester.vbus[0].indicator.led.current_limiting_resistor[Resistor:1KΩ] renamed *.tester.vbus[0].indicator.led.led[LED:D]-*.tester.vbus[0].indicator.led.current_limiting_resistor[Resistor:1.0kΩ]
- net tester.vbus[0].indicator.led[PoweredLED:virt]:2-tester.vbus[0].indicator.power_switch[PowerSwitch:vi renamed *.tester.vbus[0].indicator.led[PoweredLED:virt]:2-*.tester.vbus[0].indicator.power_switch[PowerSwitch:vi
- net tester.vbus[0][PairTester:virt]:4-tester.vbus[0].indicator[LEDIndicator:virt]-tester.vbus[0].indicat renamed *.tester.vbus[0][Pair*.tester:virt]:4-*.tester.vbus[0].indicator[LEDIndicator:virt]-*.tester.vbus[0].indicat
- net tester.vbus[1].indicator.led.led[LED:D]-tester.vbus[1].indicator.led.current_limiting_resistor[Resistor:1KΩ] renamed *.tester.vbus[1].indicator.led.led[LED:D]-*.tester.vbus[1].indicator.led.current_limiting_resistor[Resistor:1.0kΩ]
- net tester.vbus[1].indicator.power_switch[PowerSwitch:virt]:5-tester.vbus[1].indicator.led[PoweredLED:vi renamed *.tester.vbus[1].indicator.power_switch[PowerSwitch:virt]:5-*.tester.vbus[1].indicator.led[PoweredLED:vi
- net tester.vbus[1].indicator[LEDIndicator:virt]:3-tester.shield.indicator[LEDIndicator:virt]:3-tester.gn renamed *.tester.vbus[1].indicator[LEDIndicator:virt]:3-*.tester.shield.indicator[LEDIndicator:virt]:3-*.tester.gn
- net tester.vbus[1][PairTester:virt]:4-tester.vbus[1].indicator.power_switch[PowerSwitch:virt]-tester.vbu renamed *.tester.vbus[1][Pair*.tester:virt]:4-*.tester.vbus[1].indicator.power_switch[PowerSwitch:virt]-*.tester.vbu
- net tester.vbus[2].indicator.led.led[LED:D]-tester.vbus[2].indicator.led.current_limiting_resistor[Resistor:1KΩ] renamed *.tester.vbus[2].indicator.led.led[LED:D]-*.tester.vbus[2].indicator.led.current_limiting_resistor[Resistor:1.0kΩ]
- net tester.vbus[2].indicator.led[PoweredLED:virt]:2-tester.vbus[2].indicator.power_switch[PowerSwitch:vi renamed *.tester.vbus[2].indicator.led[PoweredLED:virt]:2-*.tester.vbus[2].indicator.power_switch[PowerSwitch:vi
- net tester.vbus[2][PairTester:virt]:4-tester.vbus[2].indicator[LEDIndicator:virt]-tester.vbus[2].indicat renamed *.tester.vbus[2][Pair*.tester:virt]:4-*.tester.vbus[2].indicator[LEDIndicator:virt]-*.tester.vbus[2].indicat
- net tester.vbus[3].indicator.led.current_limiting_resistor[Resistor:1KΩ]-tester.vbus[3].indicator.led.led[LED:D] renamed *.tester.vbus[3].indicator.led.current_limiting_resistor[Resistor:1.0kΩ]-*.tester.vbus[3].indicator.led.led[LED:D]
- net tester.vbus[3].indicator.power_switch[PowerSwitch:virt]:5-tester.vbus[3].indicator.led[PoweredLED:vi renamed *.tester.vbus[3].indicator.power_switch[PowerSwitch:virt]:5-*.tester.vbus[3].indicator.led[PoweredLED:vi
- net tester.vbus[3][PairTester:virt]:4-tester.vbus[3].indicator.power_switch[PowerSwitch:virt]-tester.vbu renamed *.tester.vbus[3][Pair*.tester:virt]:4-*.tester.vbus[3].indicator.power_switch[PowerSwitch:virt]-*.tester.vbu
Other:
- board text added: "USB-C Cable*.tester v1.0.1 https://github.com/IoannisP-ITENG/Cable*.tester"
- board text removed: "USB-C CableTester v1.0.1 https://github.com/IoannisP-ITENG/CableTester"
